File: 5V_ TO_3V3.kicad_sch (KiCad schematic)
At the start: 7 parts, among them U1 AP2112K-3.3

Commit message: SCHEMATIC CONTINUATION
Parts:
- renumbered C3 to C5, C4 to C6, C5 to C7, C7 to C8, C6 to C9
Connections:
- net +3V3: no longer names the net of C6.1, C7.1, U1.5 (VOUT)
- net +3V3: no longer C8.1, FB1.1
- new net: C8.1, FB1.1
Changed lines of the file:
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@@
 		)
 	)
-	(label "3V3"
-		(at 180.34 90.17 0)
+	(global_label "+5v"
+		(shape output)
+		(at 44.45 92.71 180)
+		(fields_autoplaced yes)
 		(effects
 			(font
 				(size 1.27 1.27)
 			)
-			(justify left bottom)
-		)
-	)
-	(label "3V3"
-		(at 115.57 92.71 0)
+			(justify right)
+		)
+		(property "Intersheetrefs" "${INTERSHEET_REFS}"
+			(at 37.7153 92.71 0)
+			(effects
+				(font
+					(size 1.27 1.27)
+				)
+				(justify right)
+				(hide yes)
+			)
+		)
+	)
+	(global_label "ADC-REF"
+		(shape output)
+		(at 232.41 90.17 0)
+		(fields_autoplaced yes)
 		(effects
 			(font
 				(size 1.27 1.27)
 			)
-			(justify left bottom)
-		)
-	)
-	(global_label "+5v"
+			(justify left)
+		)
+		(property "Intersheetrefs" "${INTERSHEET_REFS}"
+			(at 244.1038 90.17 0)
+			(effects
+				(font
+					(size 1.27 1.27)
+				)
+				(justify left)
+				(hide yes)
+			)
+		)
+	)
+	(global_label "3V3-EN"
 		(shape output)
-		(at 44.45 92.71 180)
+		(at 48.26 105.41 270)
 		(fields_autoplaced yes)
 		(effects
@@
 		)
 		(property "Intersheetrefs" "${INTERSHEET_REFS}"
-			(at 37.7153 92.71 0)
-			(effects
-				(font
-					(size 1.27 1.27)
-				)
-				(justify right)
-				(hide yes)
-			)
-		)
-	)
-	(global_label "+3V3"
-		(shape output)
-		(at 123.19 92.71 0)
-		(fields_autoplaced yes)
-		(effects
-			(font
-				(size 1.27 1.27)
-				(thickness 0.254)
-				(bold yes)
-			)
-			(justify left)
-		)
-		(property "Intersheetrefs" "${INTERSHEET_REFS}"
-			(at 131.7312 92.71 0)
-			(effects
-				(font
-					(size 1.27 1.27)
-				)
-				(justify left)
-				(hide yes)
-			)
-		)
-	)
-	(global_label "ADC-REF"
-		(shape output)
-		(at 232.41 90.17 0)
-		(fields_autoplaced yes)
-		(effects
-			(font
-				(size 1.27 1.27)
-			)
-			(justify left)
-		)
-		(property "Intersheetrefs" "${INTERSHEET_REFS}"
-			(at 244.1038 90.17 0)
-			(effects
-				(font
-					(size 1.27 1.27)
-				)
-				(justify left)
-				(hide yes)
-			)
-		)
-	)
-	(global_label "3V3-EN"
-		(shape output)
-		(at 48.26 105.41 270)
-		(fields_autoplaced yes)
-		(effects
-			(font
-				(size 1.27 1.27)
-			)
-			(justify right)
-		)
-		(property "Intersheetrefs" "${INTERSHEET_REFS}"
 			(at 48.26 115.9547 90)
 			(effects
@@
 		(dnp no)
 		(fields_autoplaced yes)
-		(property "Reference" "C6"
+		(property "Reference" "C9"
 			(at 215.9 99.0599 0)
 			(effects
@@
 			(project "ECM Synchronika Custom Control Board"
 				(path "/0a1cfe74-4adf-4cda-8eff-54fb631bdb34/7b9a90b3-d0b5-46b5-a44b-f4a38eaf058d"
-					(reference "C6")
+					(reference "C9")
 					(unit 1)
 				)
@@
 		(dnp no)
 		(fields_autoplaced yes)
-		(property "Reference" "#PWR07"
+		(property "Reference" "#PWR015"
 			(at 193.04 123.19 0)
 			(effects
@@
 			(project "ECM Synchronika Custom Control Board"
 				(path "/0a1cfe74-4adf-4cda-8eff-54fb631bdb34/7b9a90b3-d0b5-46b5-a44b-f4a38eaf058d"
-					(reference "#PWR07")
+					(reference "#PWR015")
 					(unit 1)
 				)
@@
 		(dnp no)
 		(fields_autoplaced yes)
-		(property "Reference" "#PWR03"
+		(property "Reference" "#PWR011"
 			(at 67.31 127 0)
 			(effects
@@
 			(project "ECM Synchronika Custom Control Board"
 				(path "/0a1cfe74-4adf-4cda-8eff-54fb631bdb34/7b9a90b3-d0b5-46b5-a44b-f4a38eaf058d"
-					(reference "#PWR03")
+					(reference "#PWR011")
 					(unit 1)
 				)
@@
 		(dnp no)
 		(fields_autoplaced yes)
-		(property "Reference" "#PWR04"
+		(property "Reference" "#PWR012"
 			(at 80.01 127 0)
 			(effects
@@
 			(project "ECM Synchronika Custom Control Board"
 				(path "/0a1cfe74-4adf-4cda-8eff-54fb631bdb34/7b9a90b3-d0b5-46b5-a44b-f4a38eaf058d"
-					(reference "#PWR04")
+					(reference "#PWR012")
 					(unit 1)
 				)
@@
 		(dnp no)
 		(fields_autoplaced yes)
-		(property "Reference" "C5"
+		(property "Reference" "C7"
 			(at 127 102.8699 0)
 			(effects
@@
 			(project "ECM Synchronika Custom Control Board"
 				(path "/0a1cfe74-4adf-4cda-8eff-54fb631bdb34/7b9a90b3-d0b5-46b5-a44b-f4a38eaf058d"
-					(reference "C5")
+					(reference "C7")
 					(unit 1)
 				)
@@
 		(dnp no)
 		(fields_autoplaced yes)
-		(property "Reference" "C4"
+		(property "Reference" "C6"
 			(at 106.68 101.5999 0)
 			(effects
@@
 			(project "ECM Synchronika Custom Control Board"
 				(path "/0a1cfe74-4adf-4cda-8eff-54fb631bdb34/7b9a90b3-d0b5-46b5-a44b-f4a38eaf058d"
-					(reference "C4")
+					(reference "C6")
 					(unit 1)
 				)
@@
 		(dnp no)
 		(fields_autoplaced yes)
-		(property "Reference" "#PWR06"
+		(property "Reference" "#PWR014"
 			(at 123.19 128.27 0)
 			(effects
@@
 			(project "ECM Synchronika Custom Control Board"
 				(path "/0a1cfe74-4adf-4cda-8eff-54fb631bdb34/7b9a90b3-d0b5-46b5-a44b-f4a38eaf058d"
-					(reference "#PWR06")
+					(reference "#PWR014")
 					(unit 1)
 				)
@@
 		(dnp no)
 		(fields_autoplaced yes)
-		(property "Reference" "C7"
+		(property "Reference" "C8"
 			(at 177.8 99.0599 0)
 			(effects
@@
 			(project "ECM Synchronika Custom Control Board"
 				(path "/0a1cfe74-4adf-4cda-8eff-54fb631bdb34/7b9a90b3-d0b5-46b5-a44b-f4a38eaf058d"
-					(reference "C7")
+					(reference "C8")
 					(unit 1)
 				)
@@
 		(on_board yes)
 		(dnp no)
-		(property "Reference" "C3"
+		(property "Reference" "C5"
 			(at 59.69 107.696 0)
 			(effects
@@
 			(project "ECM Synchronika Custom Control Board"
 				(path "/0a1cfe74-4adf-4cda-8eff-54fb631bdb34/7b9a90b3-d0b5-46b5-a44b-f4a38eaf058d"
-					(reference "C3")
+					(reference "C5")
 					(unit 1)
 				)
@@
 		(dnp no)
 		(fields_autoplaced yes)
-		(property "Reference" "#PWR05"
+		(property "Reference" "#PWR013"
 			(at 102.87 128.27 0)
 			(effects
@@
 			(project "ECM Synchronika Custom Control Board"
 				(path "/0a1cfe74-4adf-4cda-8eff-54fb631bdb34/7b9a90b3-d0b5-46b5-a44b-f4a38eaf058d"
-					(reference "#PWR05")
-					(unit 1)
-				)
+					(reference "#PWR013")
+					(unit 1)
+				)
