File: 5V_ TO_3V3.kicad_sch (KiCad schematic)
At the start: 7 parts, among them U1 AP2112K-3.3

Commit message: Update KiCad project files
Connections:
- net +3V3: now reaches C8.1, FB1.1
- net +3V3: now also C6.1, C7.1, U1.5 (VOUT)
Changed lines of the file:
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@@
+		)
+	)
+	(global_label "+3V3"
+		(shape output)
+		(at 119.38 92.71 90)
+		(fields_autoplaced yes)
+		(effects
+			(font
+				(size 1.27 1.27)
+				(thickness 0.254)
+				(bold yes)
+			)
+			(justify left)
+		)
+		(property "Intersheetrefs" "${INTERSHEET_REFS}"
+			(at 119.38 84.1688 90)
+			(effects
+				(font
+					(size 1.27 1.27)
+				)
+				(justify left)
+				(hide yes)
+			)
+		)
+	)
+	(global_label "+3V3"
+		(shape output)
+		(at 175.26 90.17 90)
+		(fields_autoplaced yes)
+		(effects
+			(font
+				(size 1.27 1.27)
+				(thickness 0.254)
+				(bold yes)
+			)
+			(justify left)
+		)
+		(property "Intersheetrefs" "${INTERSHEET_REFS}"
+			(at 175.26 81.6288 90)
+			(effects
+				(font
+					(size 1.27 1.27)
+				)
+				(justify left)
+				(hide yes)
+			)
 		)
 	)
