File: HV_INPUT .kicad_sch (KiCad schematic)
At the start: 6 parts, among them J5 Screw_Terminal_01x03

Commit message: SCHEMATIC CONTINUATION
Parts:
- renumbered C18 to C1, C20 to C2, J5 to J1
Changed lines of the file:
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@@
 		(on_board yes)
 		(dnp no)
-		(property "Reference" "C20"
+		(property "Reference" "C2"
 			(at 161.29 40.386 0)
 			(effects
@@
 			(project ""
 				(path "/0a1cfe74-4adf-4cda-8eff-54fb631bdb34/e1f8f573-d884-4909-8ded-c236ff34aedd"
-					(reference "C20")
+					(reference "C2")
 					(unit 1)
 				)
@@
 		(dnp no)
 		(fields_autoplaced yes)
-		(property "Reference" "C18"
+		(property "Reference" "C1"
 			(at 113.03 40.6399 0)
 			(effects
@@
 			(project ""
 				(path "/0a1cfe74-4adf-4cda-8eff-54fb631bdb34/e1f8f573-d884-4909-8ded-c236ff34aedd"
-					(reference "C18")
+					(reference "C1")
 					(unit 1)
 				)
@@
 		(on_board yes)
 		(dnp no)
-		(property "Reference" "J5"
+		(property "Reference" "J1"
 			(at 34.036 34.29 0)
 			(effects
@@
 			(project ""
 				(path "/0a1cfe74-4adf-4cda-8eff-54fb631bdb34/e1f8f573-d884-4909-8ded-c236ff34aedd"
-					(reference "J5")
+					(reference "J1")
 					(unit 1)
 				)
