File: HV_INPUT .kicad_sch (KiCad schematic)
At the start: 6 parts, among them J1 Screw_Terminal_01x03

Commit message: Update KiCad project files
Parts:
- removed J1: Screw_Terminal_01x03, symbol Connector:Screw_Terminal_01x03
- added J1, J6, J7: 928814-1, 6.3mm spade:TE_928814-1, symbol 6.3mm spade:928814-1
- PS1: footprint HLK-5M05:CONV_HLK-5M05 -> HLK_5M05:CONV_HLK-5M05
Connections:
- net Earth_Protective: now also J6.1
- net LIVE: now also J7.1
- net N_FUSED: now also J1.1

Commit message: Update KiCad project files
Parts:
- added C24: 100u, Capacitor_SMD:CP_Elec_6.3x5.9, symbol Device:C_Polarized
- added D17: SMBJ5.0A, SMBJ5.0A:DIOM4336X265N, symbol 5V DIODE:SMBJ5.0A
- added FB2: FerriteBead, Inductor_SMD:L_0603_1608Metric, symbol Device:FerriteBead
Connections:
- net +5v: now also C24.1, D17.C, FB2.2; no longer C2.1, PS1.4 (+VO)
- net GND: now also C24.2, D17.A
- new net: C2.1, FB2.1, PS1.4 (+VO)
Other:
- note added: "AC_INPUT_TERMINALS"

Commit message: Update KiCad project files
Parts:
- J1, J6, J7: footprint 6.3mm spade:TE_928814-1 -> 928814-1:TE_928814-1
Changed lines of the file:
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@@
-		)
-	)
-	(label "NEUTRAL"
-		(at 60.96 45.72 180)
-		(effects
-			(font
-				(size 1.27 1.27)
-			)
-			(justify right bottom)
 		)
 	)
@@
 			)
 		)
-		(property "Footprint" "6.3mm spade:TE_928814-1"
+		(property "Footprint" "928814-1:TE_928814-1"
 			(at 27.94 54.61 0)
 			(effects
@@
 			)
 		)
-		(property "Footprint" "6.3mm spade:TE_928814-1"
+		(property "Footprint" "928814-1:TE_928814-1"
 			(at 38.1 45.72 0)
 			(effects
@@
 			)
 		)
-		(property "Footprint" "6.3mm spade:TE_928814-1"
+		(property "Footprint" "928814-1:TE_928814-1"
 			(at 38.1 38.1 0)
 			(effects

Commit message: Update KiCad project files
Parts:
- removed PS1: HLK-5M05, HLK_5M05:CONV_HLK-5M05, symbol HLK-5M05:HLK-5M05
- added PS1: HLK-5M05, Converter_ACDC:Converter_ACDC_Hi-Link_HLK-5Mxx, symbol Converter_ACDC:HLK-5M05
- D17: footprint SMBJ5.0A:DIOM4336X265N -> D(5V):DIOM4336X265N
- J1, J6, J7: footprint 928814-1:TE_928814-1 -> 6.3mm spade:TE_928814-1
Connections:
- net GND: now also PS1.3 (-Vout)
- net L_FUSED: now also PS1.1 (AC/L)
- net N_FUSED: now also PS1.2 (AC/N)
- net at C2.1, FB2.1: now also PS1.4 (+Vout)
Changed lines of the file:
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@@
+	(wire
+		(pts
+			(xy 125.73 39.37) (xy 128.27 39.37)
+		)
+		(stroke
+			(width 0)
+			(type default)
+		)
+	)
 	(wire
 		(pts
@@
 	(wire
 		(pts
+			(xy 148.59 44.45) (xy 151.13 44.45)
+		)
+		(stroke
+			(width 0)
+			(type default)
+		)
+	)
+	(wire
+		(pts
 			(xy 151.13 38.1) (xy 151.13 39.37)
 		)
@@
 	(wire
 		(pts
+			(xy 125.73 44.45) (xy 128.27 44.45)
+		)
+		(stroke
+			(width 0)
+			(type default)
+		)
+	)
+	(wire
+		(pts
 			(xy 168.91 45.72) (xy 168.91 49.53)
+		)
+		(stroke
+			(width 0)
+			(type default)
+		)
+	)
+	(wire
+		(pts
+			(xy 148.59 39.37) (xy 151.13 39.37)
 		)
 		(stroke
@@
 			)
 		)
-		(property "Footprint" "928814-1:TE_928814-1"
+		(property "Footprint" "6.3mm spade:TE_928814-1"
 			(at 27.94 54.61 0)
 			(effects
@@
 			)
 		)
-		(property "Footprint" "928814-1:TE_928814-1"
+		(property "Footprint" "6.3mm spade:TE_928814-1"
 			(at 38.1 45.72 0)
 			(effects
@@
 	)
 	(symbol
+		(lib_id "Converter_ACDC:HLK-5M05")
+		(at 138.43 41.91 0)
+		(unit 1)
+		(exclude_from_sim no)
+		(in_bom yes)
+		(on_board yes)
+		(dnp no)
+		(fields_autoplaced yes)
+		(property "Reference" "PS1"
+			(at 138.43 33.02 0)
+			(effects
+				(font
+					(size 1.27 1.27)
+				)
+			)
+		)
+		(property "Value" "HLK-5M05"
+			(at 138.43 35.56 0)
+			(effects
+				(font
+					(size 1.27 1.27)
+				)
+			)
+		)
+		(property "Footprint" "Converter_ACDC:Converter_ACDC_Hi-Link_HLK-5Mxx"
+			(at 138.43 49.53 0)
+			(effects
+				(font
+					(size 1.27 1.27)
+				)
+				(hide yes)
+			)
+		)
+		(property "Datasheet" "http://h.hlktech.com/download/ACDC%E7%94%B5%E6%BA%90%E6%A8%A1%E5%9D%975W%E7%B3%BB%E5%88%97/1/%E6%B5%B7%E5%87%8C%E7%A7%915W%E7%B3%BB%E5%88%97%E7%94%B5%E6%BA%90%E6%A8%A1%E5%9D%97%E8%A7%84%E6%A0%BC%E4%B9%A6V2.8.pdf"
+			(at 148.59 52.07 0)
+			(effects
+				(font
+					(size 1.27 1.27)
+				)
+				(hide yes)
+			)
+		)
+		(property "Description" "Compact AC/DC board mount power module 5W, 5V 1A"
+			(at 138.43 41.91 0)
+			(effects
+				(font
+					(size 1.27 1.27)
+				)
+				(hide yes)
+			)
+		)
+		(pin "3"
+		)
+		(pin "1"
+		)
+		(pin "2"
+		)
+		(pin "4"
+		)
+		(instances
+			(project ""
+				(path "/0a1cfe74-4adf-4cda-8eff-54fb631bdb34/e1f8f573-d884-4909-8ded-c236ff34aedd"
+					(reference "PS1")
+					(unit 1)
+				)
+			)
+		)
+	)
+	(symbol
 		(lib_id "Device:C")
 		(at 109.22 41.91 0)
@@
 	)
 	(symbol
-		(lib_id "HLK-5M05:HLK-5M05")
-		(at 138.43 41.91 0)
-		(unit 1)
-		(exclude_from_sim no)
-		(in_bom yes)
-		(on_board yes)
-		(dnp no)
-		(property "Reference" "PS1"
-			(at 138.43 31.75 0)
-			(effects
-				(font
-					(size 1.27 1.27)
-				)
-			)
-		)
-		(property "Value" "HLK-5M05"
-			(at 138.43 34.29 0)
-			(effects
-				(font
-					(size 1.27 1.27)
-				)
-			)
-		)
-		(property "Footprint" "HLK_5M05:CONV_HLK-5M05"
-			(at 138.43 41.91 0)
-			(effects
-				(font
-					(size 1.27 1.27)
-				)
-				(justify bottom)
-				(hide yes)
-			)
-		)
-		(property "Datasheet" ""
-			(at 138.43 41.91 0)
-			(effects
-				(font
-					(size 1.27 1.27)
-				)
-				(hide yes)
-			)
-		)
-		(property "Description" ""
-			(at 138.43 41.91 0)
-			(effects
-				(font
-					(size 1.27 1.27)
-				)
-				(hide yes)
-			)
-		)
-		(property "MF" "Hi-link"
-			(at 138.43 41.91 0)
-			(effects
-				(font
-					(size 1.27 1.27)
-				)
-				(justify bottom)
-				(hide yes)
-			)
-		)
-		(property "Description_1" ""
-			(at 138.43 41.91 0)
-			(effects
-				(font
-					(size 1.27 1.27)
-				)
-				(justify bottom)
-				(hide yes)
-			)
-		)
-		(property "Package" "Package"
-			(at 138.43 41.91 0)
-			(effects
-				(font
-					(size 1.27 1.27)
-				)
-				(justify bottom)
-				(hide yes)
-			)
-		)
-		(property "Price" "None"
-			(at 138.43 41.91 0)
-			(effects
-				(font
-					(size 1.27 1.27)
-				)
-				(justify bottom)
-				(hide yes)
-			)
-		)
-		(property "Check_prices" "https://www.snapeda.com/parts/HLK-5M05/Hi-link/view-part/?ref=eda"
-			(at 138.43 41.91 0)
-			(effects
-				(font
-					(size 1.27 1.27)
-				)
-				(justify bottom)
-				(hide yes)
-			)
-		)
-		(property "STANDARD" "Manufacturer Recommendations"
-			(at 138.43 41.91 0)
-			(effects
-				(font
-					(size 1.27 1.27)
-				)
-				(justify bottom)
-				(hide yes)
-			)
-		)
-		(property "PARTREV" "N/A"
-			(at 138.43 41.91 0)
-			(effects
-				(font
-					(size 1.27 1.27)
-				)
-				(justify bottom)
-				(hide yes)
-			)
-		)
-		(property "SnapEDA_Link" "https://www.snapeda.com/parts/HLK-5M05/Hi-link/view-part/?ref=snap"
-			(at 138.43 41.91 0)
-			(effects
-				(font
-					(size 1.27 1.27)
-				)
-				(justify bottom)
-				(hide yes)
-			)
-		)
-		(property "MP" "HLK-5M05"
-			(at 138.43 41.91 0)
-			(effects
-				(font
-					(size 1.27 1.27)
-				)
-				(justify bottom)
-				(hide yes)
-			)
-		)
-		(property "Availability" "Not in stock"
-			(at 138.43 41.91 0)
-			(effects
-				(font
-					(size 1.27 1.27)
-				)
-				(justify bottom)
-				(hide yes)
-			)
-		)
-		(property "MANUFACTURER" "HI-LINK"
-			(at 138.43 41.91 0)
-			(effects
-				(font
-					(size 1.27 1.27)
-				)
-				(justify bottom)
-				(hide yes)
-			)
-		)
-		(pin "2"
-		)
-		(pin "4"
-		)
-		(pin "1"
-		)
-		(pin "3"
-		)
-		(instances
-			(project ""
-				(path "/0a1cfe74-4adf-4cda-8eff-54fb631bdb34/e1f8f573-d884-4909-8ded-c236ff34aedd"
-					(reference "PS1")
-					(unit 1)
-				)
-			)
-		)
-	)
-	(symbol
 		(lib_id "5V DIODE:SMBJ5.0A")
 		(at 194.31 44.45 90)
@@
 			)
 		)
-		(property "Footprint" "SMBJ5.0A:DIOM4336X265N"
+		(property "Footprint" "D(5V):DIOM4336X265N"
 			(at 194.31 44.45 0)
 			(effects
@@
 			)
 		)
-		(property "Footprint" "928814-1:TE_928814-1"
+		(property "Footprint" "6.3mm spade:TE_928814-1"
 			(at 38.1 38.1 0)
 			(effects

Commit message: Updated PCB files
Parts:
- removed J1, J6, J7: 928814-1, 6.3mm spade:TE_928814-1, symbol 6.3mm spade:928814-1
- added J201, J202, J203, J204, J206, J209: 928814-1, 6.3mm spade:TE_928814-1, symbol 6.3mm spade:928814-1
Connections:
- net Earth_Protective: now also J203.1
- net N_FUSED: now also J209.1
- net LIVE: no longer names the net of F1.1, RV1.1
- net LIVE: now also J201.1
- new net 3_WAY_VALVE_LOAD: J204.1
- new net LED_LOAD: J202.1
- new net PUMP_LOAD: J206.1
