File: Relays+RC SNUBBER.kicad_sch (KiCad schematic)
At the start: 32 parts, among them K1 G2RL-1-H, K3 G2RL-1-H, K5 G2RL-1-H, K6 G2RL-1-H, Q1 MMBT2222A, Q3 MMBT2222A, Q7 MMBT2222A, Q8 MMBT2222A

Commit message: SCHEMATIC CONTINUATION
Parts:
- renumbered C11 to C3, C13 to C4, D4 to D1, D13 to D2, D7 to D3, D14 to D4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
