File: Relays+RC SNUBBER.kicad_sch (KiCad schematic)
At the start: 32 parts, among them K1 G2RL-1-H, K2 G2RL-1-H, K3 G2RL-1-H, K4 G2RL-1-H, Q1 MMBT2222A, Q2 MMBT2222A, Q3 MMBT2222A, Q4 MMBT2222A

Commit message: Update KiCad project files
Parts:
- added J10, J11, J12, J13, J14, J15, J8, J9: 928814-1, 6.3mm spade:TE_928814-1, symbol 6.3mm spade:928814-1
Connections:
- net 3_WAY_VALVE_LOAD: now also J10.1
- net LED_LOAD: now also J15.1
- net L_FUSED: now also J11.1, J13.1, J14.1, J9.1
- net PUMP_LOAD: now also J8.1
- net SPARE_LOAD: now also J12.1

Commit message: Update KiCad project files
Parts:
- J10, J11, J12, J13, J14, J15, J8, J9: footprint 6.3mm spade:TE_928814-1 -> 928814-1:TE_928814-1
Connections:
- no-connect marks 0 -> 4
Changed lines of the file:
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@@
 		(color 0 0 0 0)
 	)
+	(no_connect
+		(at 48.26 44.45)
+	)
+	(no_connect
+		(at 196.85 49.53)
+	)
+	(no_connect
+		(at 48.26 130.81)
+	)
+	(no_connect
+		(at 152.4 130.81)
+	)
 	(wire
 		(pts
@@
 			)
 		)
-		(property "Footprint" "6.3mm spade:TE_928814-1"
+		(property "Footprint" "928814-1:TE_928814-1"
 			(at 33.02 152.4 0)
 			(effects
@@
 			)
 		)
-		(property "Description" "FLYBACK DIODE"
+		(property "Description" "Diode"
 			(at 76.2 144.78 0)
 			(effects
@@
 			)
 		)
-		(property "Footprint" "6.3mm spade:TE_928814-1"
+		(property "Footprint" "928814-1:TE_928814-1"
 			(at 139.7 125.73 0)
 			(effects
@@
 			)
 		)
-		(property "Description" "FLYBACK DIODE"
+		(property "Description" "Diode"
 			(at 180.34 144.78 0)
 			(effects
@@
 			)
 		)
-		(property "Footprint" "6.3mm spade:TE_928814-1"
+		(property "Footprint" "928814-1:TE_928814-1"
 			(at 35.56 39.37 0)
 			(effects
@@
 			)
 		)
-		(property "Footprint" "6.3mm spade:TE_928814-1"
+		(property "Footprint" "928814-1:TE_928814-1"
 			(at 34.29 125.73 0)
 			(effects
@@
 			)
 		)
-		(property "Footprint" "6.3mm spade:TE_928814-1"
+		(property "Footprint" "928814-1:TE_928814-1"
 			(at 24.13 67.31 0)
 			(effects
@@
 			)
 		)
-		(property "Description" "FLYBACK DIODE"
+		(property "Description" "Diode"
 			(at 76.2 58.42 0)
 			(effects
@@
 			)
 		)
-		(property "Footprint" "6.3mm spade:TE_928814-1"
+		(property "Footprint" "928814-1:TE_928814-1"
 			(at 137.16 151.13 0)
 			(effects
@@
 			)
 		)
-		(property "Footprint" "6.3mm spade:TE_928814-1"
+		(property "Footprint" "928814-1:TE_928814-1"
 			(at 185.42 69.85 0)
 			(effects
@@
 			)
 		)
-		(property "Footprint" "6.3mm spade:TE_928814-1"
+		(property "Footprint" "928814-1:TE_928814-1"
 			(at 180.34 44.45 0)
 			(effects

Commit message: Update KiCad project files
Parts:
- removed J12, J13: 928814-1, 928814-1:TE_928814-1, symbol 6.3mm spade:928814-1
- added J12: Screw_Terminal_01x03, TerminalBlock_Phoenix:TerminalBlock_Phoenix_MKDS-1,5-3-5.08_1x03_P5.08mm_Horizontal, symbol Connector:Screw_Terminal_01x03
- D1, D2, D5, D7: footprint Diode_THT:D_DO-41_SOD81_P10.16mm_Horizontal -> Diode_SMD:D_SMA
- J10, J11, J14, J15, J8, J9: footprint 928814-1:TE_928814-1 -> 6.3mm spade:TE_928814-1
- K1, K2, K3, K4: footprint Relay_THT:Relay_SPDT_Omron_G2RL-1 -> RELAY:Relay_SPDT_Omron_G2RL-1 MODIFIED
Connections:
- net L_FUSED: no longer K3.11
- net SPARE_LOAD: now also J12.2 (Pin_2)
- net at K3.12: now also J12.3 (Pin_3)
- new net: J12.1 (Pin_1), K3.11
- no-connect marks 4 -> 3
Other:
- note added: "K4 SPARE"
- note removed: "K1 SPARE"

Commit message: Updated PCB files
Parts:
- removed D5: 1N4007, Diode_SMD:D_SMA, symbol Device:D
- removed D6: LED, LED_SMD:LED_0805_2012Metric, symbol Device:LED
- removed J10, J11, J14, J15, J8, J9: 928814-1, 6.3mm spade:TE_928814-1, symbol 6.3mm spade:928814-1
- removed J12: Screw_Terminal_01x03, TerminalBlock_Phoenix:TerminalBlock_Phoenix_MKDS-1,5-3-5.08_1x03_P5.08mm_Horizontal, symbol Connector:Screw_Terminal_01x03
- removed K3: G2RL-1-H, RELAY:Relay_SPDT_Omron_G2RL-1 MODIFIED, symbol Relay:G2RL-1-H
- removed Q3: MMBT2222A, Package_TO_SOT_SMD:SOT-23, symbol Transistor_BJT:MMBT2222A
- removed R12: 10K, Resistor_SMD:R_0805_2012Metric, symbol Device:R
- removed R8: 1K, Resistor_SMD:R_0805_2012Metric, symbol Device:R
- removed R9: 470, Resistor_SMD:R_0805_2012Metric, symbol Device:R
Other:
- note removed: "K4 SPARE"
