File: SENSOR INPUT.kicad_sch (KiCad schematic)
At the start: 18 parts, among them J1 Screw_Terminal_01x02, J4 Screw_Terminal_01x03, U3 MAX31855KASA

Commit message: SCHEMATIC CONTINUATION
Parts:
- removed C2: 100n, Capacitor_SMD:C_0805_2012Metric, symbol Device:C
- removed R26: 1K, Resistor_SMD:R_0805_2012Metric, symbol Device:R
- added C13: 100n, Capacitor_SMD:C_0805_2012Metric, symbol Device:C
- added R25: 1K, Resistor_SMD:R_0805_2012Metric, symbol Device:R
- renumbered C1 to C12, C16 to C14, C17 to C16, J1 to J4, J4 to J5, R25 to R22, R27 to R26, R28 to R27
Connections:
- net at R22.1: now also R23.2, TH1.1
- net GPIO_26: now reaches R22.2
- net GPIO_26: now also C12.1, D11.1 (K)
- net ADC-REF: now reaches R23.1
- net ADC-REF: now also R24.1
- net GPIO_28: now reaches C16.1
- net GPIO_28: now also R26.2, R27.1
- net GND: now reaches C16.2
- net GND: now also C12.2, C14.2, C15.1, D11.2 (A), D12.2 (A), J5.2 (Pin_2), R27.2, TH1.2, TH2.2, U3.1 (GND), C13.2
- net T-: now reaches J4.1 (Pin_1)
- net T-: now also C14.1, U3.2 (T-)
- net T+: now reaches J4.2 (Pin_2)
- net T+: now also U3.3 (T+)
- net TRANSDUCER_SIGNAL: now reaches R26.1
- net TRANSDUCER_SIGNAL: now also J5.3 (Pin_3)
- net 3V3: now reaches U3.4 (V_{CC})
- net 3V3: now also C15.2
- net GPIO_18: now reaches U3.5 (SCK)
- net GPIO_17: now reaches U3.6 (~{CS})
- net GPIO_16: now reaches U3.7 (SO)
- net GPIO_27: now reaches D12.1 (K)
- net GPIO_27: now also C13.1, R25.2
- net at R24.2: now also TH2.1, R25.1
- net +5v: now reaches J5.1 (Pin_1)
Other:
- note added: "BREW NTC INPUT AND ESD PROTECTION"
- note added: "MAX31855KASA+_THERMOCOUPLE_INPUT"
- note added: "PRESSURE_TRANSDUCER"
- note added: "STEAM NTC INPUT AND ESD PROTECTION"
- moved on the sheet: C12, C14, C15, C16, D11, J4, J5, R22, R23, R26, R27, TH1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

Commit message: Update KiCad project files
Parts:
- added C17, C18, C19, C21, C22: 100n, Capacitor_SMD:C_0603_1608Metric, symbol Device:C
- added C20: 1u, Capacitor_SMD:C_0603_1608Metric, symbol Device:C
- added D13, D14, D15: PESD5V0S1UL, Diode_SMD:D_SOD-882, symbol Diode:PESD5V0S1UL
- added J16, J17, J18, J19, J20, J21, J22: 928814-1, 6.3mm spade:TE_928814-1, symbol 6.3mm spade:928814-1
- added R28, R29, R30, R31, R32, R33, R35: 10K, Resistor_SMD:R_0805_2012Metric, symbol Device:R
- added R34: 100, Resistor_SMD:R_0805_2012Metric, symbol Device:R
- added R36, R37: 100K, Resistor_SMD:R_0805_2012Metric, symbol Device:R
- added R38: 1M, Resistor_SMD:R_0805_2012Metric, symbol Device:R
- added U4: OPA342UA, D8, symbol OPA342UA:OPA342UA
- added U5: TLV3201AIDBVR, TLV3201AIDBVR:SOT95P280X145-5N, symbol TLV3201AIDBVR:TLV3201AIDBVR
Connections:
- net 3V3: now also C17.2, C22.2, R28.1, R29.1, R30.1, R36.1, U4.7 (V+), U5.5
- net GND: now also C17.1, C18.1, C19.1, C21.1, C22.1, D13.2 (A), D14.2 (A), D15.2 (A), J17.1, J19.1, J21.1, U4.4 (V-), U5.2
- new net: C18.2, C19.2, R31.2, R32.1
- new net: R32.2, U4.3 (IN+)
- new net: R38.1, U5.1
- new net: C21.2, R35.1, U5.3
- new net: C20.2, R34.1
- new net: R33.1, U4.2 (IN-)
- new net AC_OUT: J22.1, R31.1, R34.2, U4.6 (OUT)
- new net AC_SENSE: C20.1, R33.2, R35.2
- new net GPIO_2: D13.1 (K), J16.1, R28.2
- new net GPIO_3: D14.1 (K), J18.1, R29.2
- new net GPIO_4: R38.2
- new net GPIO_5: D15.1 (K), J20.1, R30.2
- new net V_RFE(1.65V): R36.2, R37.1, U5.4
- no-connect marks 0 -> 3
Other:
- note added: "BREW SWITCHES"
- note added: "COMPARATOR"
- note added: "DIGITAL SWITCH INPUT"
- note added: "PROBE OUTPUT"
- note added: "TANK LEVEL SWITCH"
- note added: "VOLATAGE DIVIDER TO GET 1.65V"
- note added: "WATER RESERVIOR SWITCH"
- note added: "WIEN BRIDGE OSCILLATOR"
- moved on the sheet: C12, C13, C14, C15, C16, D11, D12, J4, J5, R22, R23, R24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

Commit message: Update KiCad project files
Parts:
- J16, J17, J18, J19, J20, J21, J22: footprint 6.3mm spade:TE_928814-1 -> 928814-1:TE_928814-1
Connections:
- net GND: now also R37.2
Changed lines of the file:
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@@
 	(wire
 		(pts
-			(xy 303.53 355.6) (xy 313.69 355.6)
-		)
-		(stroke
-			(width 0)
-			(type default)
-		)
-	)
-	(wire
-		(pts
 			(xy 64.77 369.57) (xy 62.23 369.57)
 		)
@@
 	(wire
 		(pts
-			(xy 435.61 138.43) (xy 435.61 134.62)
+			(xy 303.53 355.6) (xy 307.34 355.6)
 		)
 		(stroke
@@
 	(wire
 		(pts
-			(xy 104.14 162.56) (xy 104.14 171.45)
+			(xy 435.61 138.43) (xy 435.61 134.62)
 		)
 		(stroke
@@
 	(wire
 		(pts
-			(xy 50.8 85.09) (xy 50.8 88.9)
+			(xy 104.14 162.56) (xy 104.14 171.45)
 		)
 		(stroke
@@
 	(wire
 		(pts
-			(xy 165.1 355.6) (xy 165.1 364.49)
+			(xy 50.8 85.09) (xy 50.8 88.9)
 		)
 		(stroke
@@
 	(wire
 		(pts
-			(xy 54.61 156.21) (xy 54.61 171.45)
+			(xy 165.1 355.6) (xy 165.1 364.49)
 		)
 		(stroke
@@
 	(wire
 		(pts
-			(xy 335.28 360.68) (xy 335.28 364.49)
+			(xy 54.61 156.21) (xy 54.61 171.45)
 		)
 		(stroke
@@
 	(wire
 		(pts
-			(xy 85.09 88.9) (xy 85.09 97.79)
+			(xy 335.28 360.68) (xy 335.28 364.49)
 		)
 		(stroke
@@
 	(wire
 		(pts
-			(xy 78.74 369.57) (xy 78.74 379.73)
+			(xy 85.09 88.9) (xy 85.09 97.79)
 		)
 		(stroke
@@
 	(wire
 		(pts
-			(xy 194.31 356.87) (xy 194.31 363.22)
+			(xy 78.74 369.57) (xy 78.74 379.73)
 		)
 		(stroke
@@
 		)
 	)
-	(label "WATER_SWITCH_SIGNAL"
-		(at 425.45 63.5 180)
-		(effects
-			(font
-				(size 1.27 1.27)
-				(thickness 0.254)
-				(bold yes)
-			)
-			(justify right bottom)
-		)
-	)
 	(label "AC_OUT"
 		(at 135.89 349.25 180)
@@
 		)
 	)
-	(label "BOILER"
-		(at 173.99 346.71 0)
-		(effects
-			(font
-				(size 1.27 1.27)
-				(thickness 0.254)
-				(bold yes)
-			)
-			(justify left bottom)
-		)
-	)
-	(label "BREW_HANDLE_SWITCHES"
-		(at 427.99 123.19 180)
-		(effects
-			(font
-				(size 1.27 1.27)
-				(thickness 0.254)
-				(bold yes)
-			)
-			(justify right bottom)
-		)
-	)
 	(label "T+"
 		(at 71.12 213.36 0)
@@
 		)
 	)
-	(label "TANK_LEVEL_SIGNAL"
-		(at 515.62 63.5 180)
-		(effects
-			(font
-				(size 1.27 1.27)
-				(thickness 0.254)
-				(bold yes)
-			)
-			(justify right bottom)
-		)
-	)
 	(label "AC_SENSE"
 		(at 234.95 358.14 180)
@@
 		)
 	)
-	(label "BOILER_BODY"
-		(at 194.31 356.87 0)
-		(effects
-			(font
-				(size 1.27 1.27)
-				(thickness 0.254)
-				(bold yes)
-			)
-			(justify left bottom)
-		)
-	)
 	(label "AC_SENSE"
 		(at 161.29 378.46 180)
@@
 			)
 		)
-		(property "Footprint" "6.3mm spade:TE_928814-1"
+		(property "Footprint" "928814-1:TE_928814-1"
 			(at 394.97 63.5 0)
 			(effects
@@
 			)
 		)
-		(property "Footprint" "6.3mm spade:TE_928814-1"
+		(property "Footprint" "928814-1:TE_928814-1"
 			(at 194.31 346.71 0)
 			(effects
@@
 	(symbol
 		(lib_id "power:GND")
+		(at 335.28 375.92 0)
+		(unit 1)
+		(exclude_from_sim no)
+		(in_bom yes)
+		(on_board yes)
+		(dnp no)
+		(fields_autoplaced yes)
+		(property "Reference" "#PWR049"
+			(at 335.28 382.27 0)
+			(effects
+				(font
+					(size 1.27 1.27)
+				)
+				(hide yes)
+			)
+		)
+		(property "Value" "GND"
+			(at 335.28 381 0)
+			(effects
+				(font
+					(size 1.27 1.27)
+				)
+			)
+		)
+		(property "Footprint" ""
+			(at 335.28 375.92 0)
+			(effects
+				(font
+					(size 1.27 1.27)
+				)
+				(hide yes)
+			)
+		)
+		(property "Datasheet" ""
+			(at 335.28 375.92 0)
+			(effects
+				(font
+					(size 1.27 1.27)
+				)
+				(hide yes)
+			)
+		)
+		(property "Description" "Power symbol creates a global label with name \"GND\" , ground"
+			(at 335.28 375.92 0)
+			(effects
+				(font
+					(size 1.27 1.27)
+				)
+				(hide yes)
+			)
+		)
+		(pin "1"
+		)
+		(instances
+			(project "ECM Synchronika Custom Control Board"
+				(path "/0a1cfe74-4adf-4cda-8eff-54fb631bdb34/219dc6f5-caa4-4fbf-9730-f96a4d06b3e9"
+					(reference "#PWR049")
+					(unit 1)
+				)
+			)
+		)
+	)
+	(symbol
+		(lib_id "power:GND")
 		(at 109.22 54.61 0)
 		(unit 1)
@@
 			)
 		)
-		(property "Footprint" "6.3mm spade:TE_928814-1"
+		(property "Footprint" "928814-1:TE_928814-1"
 			(at 394.97 78.74 0)
 			(effects
@@
 			)
 		)
-		(property "Footprint" "6.3mm spade:TE_928814-1"
+		(property "Footprint" "928814-1:TE_928814-1"
 			(at 485.14 63.5 0)
 			(effects
@@
 			)
 		)
-		(property "Footprint" "6.3mm spade:TE_928814-1"
+		(property "Footprint" "928814-1:TE_928814-1"
 			(at 397.51 138.43 0)
 			(effects
@@
 			)
 		)
-		(property "Footprint" "6.3mm spade:TE_928814-1"
+		(property "Footprint" "928814-1:TE_928814-1"
 			(at 485.14 78.74 0)
 			(effects
@@
 			)
 		)
-		(property "Footprint" "6.3mm spade:TE_928814-1"
+		(property "Footprint" "928814-1:TE_928814-1"
 			(at 397.51 123.19 0)
 			(effects
@@
 					(unit 1)
 				)
-			)
-		)
-	)
-	(symbol
-		(lib_id "power:Earth_Protective")
-		(at 194.31 363.22 0)
-		(mirror y)
-		(unit 1)
-		(exclude_from_sim no)
-		(in_bom yes)
-		(on_board yes)
-		(dnp no)
-		(property "Reference" "#PWR036"
-			(at 194.31 373.38 0)
-			(effects
-				(font
-					(size 1.27 1.27)
-				)
-				(hide yes)
-			)
-		)
-		(property "Value" "Earth_Protective"
-			(at 194.31 372.11 0)
-			(effects
-				(font
-					(size 1.27 1.27)
-				)
-			)
-		)
-		(property "Footprint" ""
-			(at 194.31 365.76 0)
-			(effects
-				(font
-					(size 1.27 1.27)
-				)
-				(hide yes)
-			)
-		)
-		(property "Datasheet" "~"
-			(at 194.31 365.76 0)
-			(effects
-				(font
-					(size 1.27 1.27)
-				)
-				(hide yes)
-			)
-		)
-		(property "Description" "Power symbol creates a global label with name \"Earth_Protective\""
-			(at 194.31 363.22 0)
-			(effects
-				(font
-					(size 1.27 1.27)
-				)
-				(hide yes)
-			)
-		)
-		(pin "1"
-		)
-		(instances
-			(project "ECM Synchronika Custom Control Board"
-				(path "/0a1cfe74-4adf-4cda-8eff-54fb631bdb34/219dc6f5-caa4-4fbf-9730-f96a4d06b3e9"
-					(reference "#PWR036")
-					(unit 1)
-				)

Commit message: Update KiCad project files
Parts:
- J16, J17, J18, J19, J20, J21, J22: footprint 928814-1:TE_928814-1 -> 6.3mm spade:TE_928814-1
- U4: footprint D8 -> OPA342UA:D8
- U5: footprint TLV3201AIDBVR:SOT95P280X145-5N -> COMPARATOR:COMPARTOR_SOT95P280X145-5N
Connections:
- net GND: no longer C12.2, C13.2, C14.2, C15.1, D11.2 (A), D12.2 (A), TH1.2, TH2.2, U3.1 (GND)
- net 3V3 renamed +3V3
- new net GNDA: C12.2, C13.2, C14.2, C15.1, D11.2 (A), D12.2 (A), TH1.2, TH2.2, U3.1 (GND)

Commit message: Update KiCad project files
Parts:
- removed J4: Screw_Terminal_01x02, TerminalBlock_Phoenix:TerminalBlock_Phoenix_MKDS-1,5-2-5.08_1x02_P5.08mm_Horizontal, symbol Connector:Screw_Terminal_01x02
- removed J5: Screw_Terminal_01x03, TerminalBlock_Phoenix:TerminalBlock_Phoenix_MKDS-1,5-3-5.08_1x03_P5.08mm_Horizontal, symbol Connector:Screw_Terminal_01x03
Connections:
- net T+ renamed THERMOCOUPLE+
- net T- renamed THERMOCOUPLE-
- net TRANSDUCER_SIGNAL renamed PRESSUE-SIGNAL
