File: SENSOR INPUT.kicad_sch (KiCad schematic)
At the start: 45 parts, among them J16 928814-1, J17 928814-1, J18 928814-1, J19 928814-1, J20 928814-1, J21 928814-1, J22 928814-1, U3 MAX31855KASA, U4 OPA342UA, U5 TLV3201AIDBVR

Commit message: Updated PCB files
Parts:
- removed J16, J17, J18, J19, J20, J21, J22: 928814-1, 6.3mm spade:TE_928814-1, symbol 6.3mm spade:928814-1
- added J702: Screw_Terminal_01x06, TerminalBlock_Phoenix:TerminalBlock_Phoenix_MPT-0,5-6-2.54_1x06_P2.54mm_Horizontal, symbol Connector:Screw_Terminal_01x06
- added J703: Screw_Terminal_01x12, TerminalBlock_Phoenix:TerminalBlock_Phoenix_MPT-0,5-12-2.54_1x12_P2.54mm_Horizontal, symbol Connector:Screw_Terminal_01x12
Connections:
- net AC_OUT: now also J702.6 (Pin_6)
- net GND: now also J702.2 (Pin_2), J702.4 (Pin_4), J703.12 (Pin_12), J703.2 (Pin_2)
- net GPIO_2: now also J702.5 (Pin_5)
- net GPIO_3: now also J702.3 (Pin_3)
- net GPIO_5: now also J702.1 (Pin_1)
- net PRESSUE-SIGNAL: now also J703.1 (Pin_1)
- net THERMOCOUPLE+: now also J703.4 (Pin_4)
- net THERMOCOUPLE-: now also J703.5 (Pin_5)
- new net +5v: J703.3 (Pin_3), J703.7 (Pin_7), J703.9 (Pin_9)
- new net BREW_HEATER_-(C): J703.6 (Pin_6)
- new net CT_LINE+: J703.10 (Pin_10)
- new net CT_LINE-: J703.11 (Pin_11)
- new net STEAM_HEATER_-(C): J703.8 (Pin_8)
