File: SSR.kicad_sch (KiCad schematic)
At the start: 12 parts, among them J2 Screw_Terminal_01x02, J3 Screw_Terminal_01x02, Q5 MMBT2222A, Q6 MMBT2222A

Commit message: SCHEMATIC CONTINUATION
Parts:
- removed R22: 10K, Resistor_SMD:R_0805_2012Metric, symbol Device:R
- added R19: 1K, Resistor_SMD:R_0805_2012Metric, symbol Device:R
- R20: value 1K -> 10K
- renumbered R17 to R16, R18 to R17, R19 to R18
Connections:
- net at D10.1 (K): now also R21.2
- net SSR_INPUT_-: now reaches D10.2 (A)
- net SSR_INPUT_-: now also D9.2 (A), J2.2 (Pin_2), J3.2 (Pin_2), Q5.3 (C), Q6.3 (C)
- net GPIO_13: now reaches R16.1
- net at R16.2: now also Q5.1 (B), R17.1
- net +5v: now reaches R21.1
- net +5v: now also J2.1 (Pin_1), J3.1 (Pin_1), R18.1
- net at Q6.1 (B): now also R20.1, R19.2
- net GND: now reaches Q6.2 (E)
- net GND: now also Q5.2 (E), R17.2, R20.2
- net at R18.2: now also D9.1 (K)
- new net GPIO_14: R19.1
Other:
- note added: "BREW HEATER"
- note added: "STEAM HEATER"
- moved on the sheet: D9, J2, Q5, R16, R17, R18

Commit message: Update KiCad project files
Changed lines of the file:
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@@
-		)
-	)
-	(label "SSR_INPUT_+"
-		(at 158.75 59.69 0)
-		(effects
-			(font
-				(size 1.27 1.27)
-			)
-			(justify left bottom)
-		)
-	)
-	(label "SSR_INPUT_+"
-		(at 41.91 60.96 0)
-		(effects
-			(font
-				(size 1.27 1.27)
-			)
-			(justify left bottom)
 		)
 	)

Commit message: Update KiCad project files
Parts:
- J2, J3: footprint TerminalBlock_Phoenix:TerminalBlock_Phoenix_MKDS-1-2-3.81_1x02_P3.81mm_Horizontal -> TerminalBlock_Phoenix:TerminalBlock_Phoenix_MKDS-3-2-5.08_1x02_P5.08mm_Horizontal
Connections:
- net SSR_INPUT_-: no longer names the net of D10.2 (A), J3.2 (Pin_2), Q6.3 (C)
- net SSR_INPUT_-: no longer D9.2 (A), J2.2 (Pin_2), Q5.3 (C)
- new net: D9.2 (A), J2.2 (Pin_2), Q5.3 (C)
Changed lines of the file:
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@@
-		)
-	)
-	(label "SSR_INPUT_-"
-		(at 41.91 86.36 0)
-		(effects
-			(font
-				(size 1.27 1.27)
-			)
-			(justify left bottom)
-		)
-	)
-	(label "SSR_INPUT_-"
-		(at 163.83 85.09 0)
-		(effects
-			(font
-				(size 1.27 1.27)
-			)
-			(justify left bottom)
 		)
 	)
@@
 			)
 		)
-		(property "Footprint" "TerminalBlock_Phoenix:TerminalBlock_Phoenix_MKDS-1-2-3.81_1x02_P3.81mm_Horizontal"
+		(property "Footprint" "TerminalBlock_Phoenix:TerminalBlock_Phoenix_MKDS-3-2-5.08_1x02_P5.08mm_Horizontal"
 			(at 151.13 69.85 0)
 			(effects
@@
 			)
 		)
-		(property "Footprint" "TerminalBlock_Phoenix:TerminalBlock_Phoenix_MKDS-1-2-3.81_1x02_P3.81mm_Horizontal"
+		(property "Footprint" "TerminalBlock_Phoenix:TerminalBlock_Phoenix_MKDS-3-2-5.08_1x02_P5.08mm_Horizontal"
 			(at 31.75 71.12 0)
 			(effects

Commit message: Update KiCad project files
Parts:
- removed J2, J3: Screw_Terminal_01x02, TerminalBlock_Phoenix:TerminalBlock_Phoenix_MKDS-3-2-5.08_1x02_P5.08mm_Horizontal, symbol Connector:Screw_Terminal_01x02
Connections:
- net STEAM_HEATER_-(C): now reaches D10.2 (A), Q6.3 (C)
- net BREW_HEATER_-(C): now reaches D9.2 (A), Q5.3 (C)
Changed lines of the file:
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@@
+	)
+	(junction
+		(at 184.15 85.09)
+		(diameter 0)
+		(color 0 0 0 0)
+	)
+	(junction
+		(at 167.64 99.06)
+		(diameter 0)
+		(color 0 0 0 0)
 	)
 	(junction
@@
 		(color 0 0 0 0)
 	)
-	(junction
-		(at 167.64 99.06)
-		(diameter 0)
-		(color 0 0 0 0)
-	)
-	(junction
-		(at 184.15 85.09)
-		(diameter 0)
-		(color 0 0 0 0)
+	(wire
+		(pts
+			(xy 62.23 60.96) (xy 92.71 60.96)
+		)
+		(stroke
+			(width 0)
+			(type default)
+		)
 	)
 	(wire
@@
 	(wire
 		(pts
-			(xy 36.83 60.96) (xy 92.71 60.96)
-		)
-		(stroke
-			(width 0)
-			(type default)
-		)
-	)
-	(wire
-		(pts
-			(xy 156.21 72.39) (xy 156.21 85.09)
-		)
-		(stroke
-			(width 0)
-			(type default)
-		)
-	)
-	(wire
-		(pts
-			(xy 36.83 73.66) (xy 36.83 86.36)
-		)
-		(stroke
-			(width 0)
-			(type default)
-		)
-	)
-	(wire
-		(pts
-			(xy 36.83 71.12) (xy 36.83 60.96)
+			(xy 181.61 59.69) (xy 212.09 59.69)
+		)
+		(stroke
+			(width 0)
+			(type default)
+		)
+	)
+	(wire
+		(pts
+			(xy 171.45 85.09) (xy 184.15 85.09)
 		)
 		(stroke
@@
 	(wire
 		(pts
+			(xy 44.45 86.36) (xy 64.77 86.36)
+		)
+		(stroke
+			(width 0)
+			(type default)
+		)
+	)
+	(wire
+		(pts
 			(xy 184.15 85.09) (xy 212.09 85.09)
 		)
@@
 	(wire
 		(pts
-			(xy 36.83 86.36) (xy 64.77 86.36)
-		)
-		(stroke
-			(width 0)
-			(type default)
-		)
-	)
-	(wire
-		(pts
 			(xy 149.86 99.06) (xy 153.67 99.06)
 		)
@@
 	(wire
 		(pts
-			(xy 156.21 85.09) (xy 184.15 85.09)
-		)
-		(stroke
-			(width 0)
-			(type default)
-		)
-	)
-	(wire
-		(pts
-			(xy 156.21 59.69) (xy 212.09 59.69)
-		)
-		(stroke
-			(width 0)
-			(type default)
-		)
-	)
-	(wire
-		(pts
-			(xy 212.09 66.04) (xy 212.09 59.69)
-		)
-		(stroke
-			(width 0)
-			(type default)
-		)
-	)
-	(wire
-		(pts
-			(xy 156.21 69.85) (xy 156.21 59.69)
+			(xy 212.09 59.69) (xy 212.09 66.04)
 		)
 		(stroke
@@
 	(wire
 		(pts
-			(xy 92.71 67.31) (xy 92.71 60.96)
-		)
-		(stroke
-			(width 0)
-			(type default)
+			(xy 92.71 60.96) (xy 92.71 67.31)
+		)
+		(stroke
+			(width 0)
+			(type default)
+		)
+	)
+	(global_label "STEAM_HEATER_-(C)"
+		(shape input)
+		(at 171.45 85.09 90)
+		(fields_autoplaced yes)
+		(effects
+			(font
+				(size 1.27 1.27)
+				(thickness 0.254)
+				(bold yes)
+			)
+			(justify left)
+		)
+		(property "Intersheetrefs" "${INTERSHEET_REFS}"
+			(at 171.45 62.337 90)
+			(effects
+				(font
+					(size 1.27 1.27)
+				)
+				(justify left)
+				(hide yes)
+			)
 		)
 	)
@@
 		)
 	)
+	(global_label "BREW_HEATER_-(C)"
+		(shape input)
+		(at 44.45 86.36 90)
+		(fields_autoplaced yes)
+		(effects
+			(font
+				(size 1.27 1.27)
+				(thickness 0.254)
+				(bold yes)
+			)
+			(justify left)
+		)
+		(property "Intersheetrefs" "${INTERSHEET_REFS}"
+			(at 44.45 64.3327 90)
+			(effects
+				(font
+					(size 1.27 1.27)
+				)
+				(justify left)
+				(hide yes)
+			)
+		)
+	)
 	(global_label "+5v"
 		(shape input)
@@
 			)
 			(justify right)
-		)
-	)
-	(symbol
-		(lib_id "Connector:Screw_Terminal_01x02")
-		(at 151.13 69.85 0)
-		(mirror y)
-		(unit 1)
-		(exclude_from_sim no)
-		(in_bom yes)
-		(on_board yes)
-		(dnp no)
-		(property "Reference" "J3"
-			(at 148.59 69.8499 0)
-			(effects
-				(font
-					(size 1.27 1.27)
-				)
-				(justify left)
-			)
-		)
-		(property "Value" "Screw_Terminal_01x02"
-			(at 143.256 84.074 90)
-			(effects
-				(font
-					(size 1.27 1.27)
-				)
-				(justify left)
-			)
-		)
-		(property "Footprint" "TerminalBlock_Phoenix:TerminalBlock_Phoenix_MKDS-3-2-5.08_1x02_P5.08mm_Horizontal"
-			(at 151.13 69.85 0)
-			(effects
-				(font
-					(size 1.27 1.27)
-				)
-				(hide yes)
-			)
-		)
-		(property "Datasheet" "~"
-			(at 151.13 69.85 0)
-			(effects
-				(font
-					(size 1.27 1.27)
-				)
-				(hide yes)
-			)
-		)
-		(property "Description" "Generic screw terminal, single row, 01x02, script generated (kicad-library-utils/schlib/autogen/connector/)"
-			(at 151.13 69.85 0)
-			(effects
-				(font
-					(size 1.27 1.27)
-				)
-				(hide yes)
-			)
-		)
-		(pin "2"
-		)
-		(pin "1"
-		)
-		(instances
-			(project "ECM Synchronika Custom Control Board"
-				(path "/0a1cfe74-4adf-4cda-8eff-54fb631bdb34/66e61237-0dee-4721-9e95-e23431ee422c"
-					(reference "J3")
-					(unit 1)
-				)
-			)
 		)
 	)
@@
 					(unit 1)
 				)
-			)
-		)
-	)
-	(symbol
-		(lib_id "Connector:Screw_Terminal_01x02")
-		(at 31.75 71.12 0)
-		(mirror y)
-		(unit 1)
-		(exclude_from_sim no)
-		(in_bom yes)
-		(on_board yes)
-		(dnp no)
-		(property "Reference" "J2"
-			(at 29.21 71.1199 0)
-			(effects
-				(font
-					(size 1.27 1.27)
-				)
-				(justify left)
-			)
-		)
-		(property "Value" "Screw_Terminal_01x02"
-			(at 23.876 85.09 90)
-			(effects
-				(font
-					(size 1.27 1.27)
-				)
-				(justify left)
-			)
-		)
-		(property "Footprint" "TerminalBlock_Phoenix:TerminalBlock_Phoenix_MKDS-3-2-5.08_1x02_P5.08mm_Horizontal"
-			(at 31.75 71.12 0)
-			(effects
-				(font
-					(size 1.27 1.27)
-				)
-				(hide yes)
-			)
-		)
-		(property "Datasheet" "~"
-			(at 31.75 71.12 0)
-			(effects
-				(font
-					(size 1.27 1.27)
-				)
-				(hide yes)
-			)
-		)
-		(property "Description" "Generic screw terminal, single row, 01x02, script generated (kicad-library-utils/schlib/autogen/connector/)"
-			(at 31.75 71.12 0)
-			(effects
-				(font
-					(size 1.27 1.27)
-				)
-				(hide yes)
-			)
-		)
-		(pin "2"
-		)
-		(pin "1"
-		)
-		(instances
-			(project ""
-				(path "/0a1cfe74-4adf-4cda-8eff-54fb631bdb34/66e61237-0dee-4721-9e95-e23431ee422c"
-					(reference "J2")
-					(unit 1)
-				)
