File: ECM Synchronika Custom Control Board.kicad_sch (KiCad schematic)
At the start: 0 parts

Commit message: SCHEMATIC CONTINUATION
Other:
- sheet MCU ports: added GPIO_10, GPIO_11, GPIO_12, GPIO_13, GPIO_14, GPIO_20; removed none
- sheet SSR ports: added GPIO_13, GPIO_14; removed none
Changed lines of the file:
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@@
+	(wire
+		(pts
+			(xy 82.55 25.4) (xy 96.52 25.4)
+		)
+		(stroke
+			(width 0)
+			(type default)
+		)
+	)
+	(wire
+		(pts
+			(xy 82.55 35.56) (xy 96.52 35.56)
+		)
+		(stroke
+			(width 0)
+			(type default)
+		)
+	)
+	(wire
+		(pts
+			(xy 125.73 24.13) (xy 135.89 24.13)
+		)
+		(stroke
+			(width 0)
+			(type default)
+		)
+	)
+	(wire
+		(pts
+			(xy 82.55 30.48) (xy 96.52 30.48)
+		)
+		(stroke
+			(width 0)
+			(type default)
+		)
+	)
+	(wire
+		(pts
+			(xy 82.55 20.32) (xy 96.52 20.32)
+		)
+		(stroke
+			(width 0)
+			(type default)
+		)
+	)
 	(wire
 		(pts
 			(xy 40.64 33.02) (xy 53.34 33.02)
+		)
+		(stroke
+			(width 0)
+			(type default)
+		)
+	)
+	(wire
+		(pts
+			(xy 125.73 19.05) (xy 135.89 19.05)
 		)
 		(stroke
@@
 		)
 		(pin "GPIO_10" output
-			(at 82.55 20.955 0)
+			(at 82.55 20.32 0)
 			(effects
 				(font
@@
 		)
 		(pin "GPIO_11" output
-			(at 82.55 26.035 0)
+			(at 82.55 25.4 0)
 			(effects
 				(font
@@
 		)
 		(pin "GPIO_20" output
-			(at 82.55 31.115 0)
+			(at 82.55 30.48 0)
 			(effects
 				(font
@@
 	)
 	(sheet
-		(at 234.95 16.51)
-		(size 27.94 20.32)
+		(at 135.89 16.51)
+		(size 27.94 19.685)
 		(exclude_from_sim no)
 		(in_bom yes)
@@
 		)
 		(property "Sheetname" "SSR"
-			(at 234.95 15.7984 0)
+			(at 135.89 15.7984 0)
 			(effects
 				(font
@@
 		)
 		(property "Sheetfile" "SSR.kicad_sch"
-			(at 234.95 37.4146 0)
-			(effects
-				(font
-					(size 1.27 1.27)
-				)
-				(justify left top)
+			(at 135.89 36.7796 0)
+			(effects
+				(font
+					(size 1.27 1.27)
+				)
+				(justify left top)
+			)
+		)
+		(pin "GPIO_13" input
+			(at 135.89 19.05 180)
+			(effects
+				(font
+					(size 1.27 1.27)
+				)
+				(justify left)
+			)
+		)
+		(pin "GPIO_14" input
+			(at 135.89 24.13 180)
+			(effects
+				(font
+					(size 1.27 1.27)
+				)
+				(justify left)
 			)
 		)
@@
 	)
 	(sheet
-		(at 139.7 14.605)
+		(at 172.72 15.875)
 		(size 27.94 20.32)
 		(exclude_from_sim no)
@@
 		)
 		(property "Sheetname" "5V_ TO_3V3"
-			(at 139.7 13.8934 0)
+			(at 172.72 15.1634 0)
 			(effects
 				(font
@@
 		)
 		(property "Sheetfile" "5V_ TO_3V3.kicad_sch"
-			(at 139.7 35.5096 0)
+			(at 172.72 36.7796 0)
 			(effects
 				(font
@@
 	)
 	(sheet
-		(at 94.615 16.51)
-		(size 29.21 20.32)
+		(at 96.52 16.51)
+		(size 29.21 20.955)
 		(exclude_from_sim no)
 		(in_bom yes)
@@
 		)
 		(property "Sheetname" "MCU"
-			(at 94.615 15.7984 0)
+			(at 96.52 15.7984 0)
 			(effects
 				(font
@@
 		)
 		(property "Sheetfile" "MCU.kicad_sch"
-			(at 94.615 37.4146 0)
-			(effects
-				(font
-					(size 1.27 1.27)
-				)
-				(justify left top)
-			)
-		)
+			(at 96.52 38.0496 0)
+			(effects
+				(font
+					(size 1.27 1.27)
+				)
+				(justify left top)
+			)
+		)
+		(pin "GPIO_10" output
+			(at 96.52 20.32 180)
+			(effects
+				(font
+					(size 1.27 1.27)
+				)
+				(justify left)
+			)
+		)
+		(pin "GPIO_11" output
+			(at 96.52 25.4 180)
+			(effects
+				(font
+					(size 1.27 1.27)
+				)
+				(justify left)
+			)
+		)
+		(pin "GPIO_12" output
+			(at 96.52 35.56 180)
+			(effects
+				(font
+					(size 1.27 1.27)
+				)
+				(justify left)
+			)
+		)
+		(pin "GPIO_20" output
+			(at 96.52 30.48 180)
+			(effects
+				(font
+					(size 1.27 1.27)
+				)
+				(justify left)
+			)
+		)
+		(pin "GPIO_13" input
+			(at 125.73 19.05 0)
+			(effects
+				(font
+					(size 1.27 1.27)
+				)
+				(justify right)
+			)
+		)
+		(pin "GPIO_14" input
+			(at 125.73 24.13 0)
+			(effects
+				(font
+					(size 1.27 1.27)
+				)
+				(justify right)
+			)
+		)

Commit message: Update KiCad project files
Other:
- sheet SENSOR INPUT ports: added GPIO_16, GPIO_17, GPIO_18, GPIO_26, GPIO_27, GPIO_28; removed none
Changed lines of the file:
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@@
+			)
+		)
+		(pin "GPIO_16" input
+			(at 57.15 92.71 0)
+			(effects
+				(font
+					(size 1.27 1.27)
+				)
+				(justify right)
+			)
+		)
+		(pin "GPIO_17" input
+			(at 57.15 96.52 0)
+			(effects
+				(font
+					(size 1.27 1.27)
+				)
+				(justify right)
+			)
+		)
+		(pin "GPIO_18" input
+			(at 57.15 100.33 0)
+			(effects
+				(font
+					(size 1.27 1.27)
+				)
+				(justify right)
+			)
+		)
+		(pin "GPIO_26" input
+			(at 57.15 104.14 0)
+			(effects
+				(font
+					(size 1.27 1.27)
+				)
+				(justify right)
+			)
+		)
+		(pin "GPIO_27" input
+			(at 57.15 106.68 0)
+			(effects
+				(font
+					(size 1.27 1.27)
+				)
+				(justify right)
+			)
+		)
+		(pin "GPIO_28" input
+			(at 57.15 88.9 0)
+			(effects
+				(font
+					(size 1.27 1.27)
+				)
+				(justify right)
 			)
 		)

Commit message: Update KiCad project files
Other:
- added sheet PORTS (PORTS.kicad_sch)
- sheet SENSOR INPUT ports: added GPIO_2, GPIO_3, GPIO_4, GPIO_5; removed none
Changed lines of the file:
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@@
+	)
+	(sheet
+		(at 90.17 62.23)
+		(size 36.83 26.67)
+		(exclude_from_sim no)
+		(in_bom yes)
+		(on_board yes)
+		(dnp no)
+		(fields_autoplaced yes)
+		(stroke
+			(width 0.1524)
+			(type solid)
+		)
+		(fill
+			(color 0 0 0 0.0000)
+		)
+		(property "Sheetname" "PORTS"
+			(at 90.17 61.5184 0)
+			(effects
+				(font
+					(size 1.27 1.27)
+				)
+				(justify left bottom)
+			)
+		)
+		(property "Sheetfile" "PORTS.kicad_sch"
+			(at 90.17 89.4846 0)
+			(effects
+				(font
+					(size 1.27 1.27)
+				)
+				(justify left top)
+			)
+		)
+		(instances
+			(project "ECM Synchronika Custom Control Board"
+				(path "/0a1cfe74-4adf-4cda-8eff-54fb631bdb34"
+					(page "8")
+				)
+			)
+		)
 	)
 	(sheet
@@
 			)
 		)
+		(pin "GPIO_2" input
+			(at 30.48 92.71 180)
+			(effects
+				(font
+					(size 1.27 1.27)
+				)
+				(justify left)
+			)
+		)
+		(pin "GPIO_3" input
+			(at 30.48 97.79 180)
+			(effects
+				(font
+					(size 1.27 1.27)
+				)
+				(justify left)
+			)
+		)
+		(pin "GPIO_4" input
+			(at 30.48 101.6 180)
+			(effects
+				(font
+					(size 1.27 1.27)
+				)
+				(justify left)
+			)
+		)
+		(pin "GPIO_5" input
+			(at 30.48 105.41 180)
+			(effects
+				(font
+					(size 1.27 1.27)
+				)
+				(justify left)
+			)
+		)

Commit message: Update KiCad project files
Other:
- sheet MCU ports: added GPIO6, GPIO7, GPIO_16, GPIO_17, GPIO_18, GPIO_2, GPIO_26, GPIO_27, GPIO_28, GPIO_3, GPIO_4, GPIO_5; removed none
- sheet PORTS ports: added GPIO6, GPIO7, L_FUSED, N_FUSED; removed none

Commit message: Update KiCad project files
Parts:
- added H1: MountingHole_Pad, MountingHole:MountingHole_3.2mm_M3_ISO7380_Pad_TopBottom, symbol Mechanical:MountingHole_Pad
- added H2, H3, H4: MountingHole, MountingHole:MountingHole_3.2mm_M3_ISO14580, symbol Mechanical:MountingHole
Connections:
- new net Earth_Protective: H1.1
Other:
- sheet MCU renamed MCU (page 4)

Commit message: Update KiCad project files
Other:
- sheet PORTS ports: added GPIO_26, GPIO_27, GPIO_28; removed none
Changed lines of the file:
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@@
 	(paper "A4")
+	(junction
+		(at 91.44 17.78)
+		(diameter 0)
+		(color 0 0 0 0)
+	)
 	(junction
 		(at 40.64 33.02)
@@
 		(color 0 0 0 0)
 	)
+	(junction
+		(at 139.7 20.32)
+		(diameter 0)
+		(color 0 0 0 0)
+	)
+	(junction
+		(at 135.89 17.78)
+		(diameter 0)
+		(color 0 0 0 0)
+	)
 	(wire
 		(pts
@@
 	(wire
 		(pts
+			(xy 39.37 73.66) (xy 91.44 73.66)
+		)
+		(stroke
+			(width 0)
+			(type default)
+		)
+	)
+	(wire
+		(pts
 			(xy 110.49 -30.48) (xy 110.49 -39.37)
 		)
@@
 	(wire
 		(pts
+			(xy 115.57 36.83) (xy 115.57 59.69)
+		)
+		(stroke
+			(width 0)
+			(type default)
+		)
+	)
+	(wire
+		(pts
+			(xy 82.55 25.4) (xy 96.52 25.4)
+		)
+		(stroke
+			(width 0)
+			(type default)
+		)
+	)
+	(wire
+		(pts
+			(xy 110.49 -39.37) (xy 168.91 -39.37)
+		)
+		(stroke
+			(width 0)
+			(type default)
+		)
+	)
+	(wire
+		(pts
+			(xy 168.91 59.69) (xy 115.57 59.69)
+		)
+		(stroke
+			(width 0)
+			(type default)
+		)
+	)
+	(wire
+		(pts
+			(xy 21.59 97.79) (xy 21.59 137.16)
+		)
+		(stroke
+			(width 0)
+			(type default)
+		)
+	)
+	(wire
+		(pts
+			(xy 82.55 35.56) (xy 96.52 35.56)
+		)
+		(stroke
+			(width 0)
+			(type default)
+		)
+	)
+	(wire
+		(pts
 			(xy 135.89 1.27) (xy 135.89 17.78)
 		)
@@
 	(wire
 		(pts
-			(xy 115.57 36.83) (xy 115.57 59.69)
-		)
-		(stroke
-			(width 0)
-			(type default)
-		)
-	)
-	(wire
-		(pts
-			(xy 82.55 25.4) (xy 96.52 25.4)
-		)
-		(stroke
-			(width 0)
-			(type default)
-		)
-	)
-	(wire
-		(pts
-			(xy 110.49 -39.37) (xy 168.91 -39.37)
-		)
-		(stroke
-			(width 0)
-			(type default)
-		)
-	)
-	(wire
-		(pts
-			(xy 168.91 59.69) (xy 115.57 59.69)
-		)
-		(stroke
-			(width 0)
-			(type default)
-		)
-	)
-	(wire
-		(pts
-			(xy 21.59 97.79) (xy 21.59 137.16)
-		)
-		(stroke
-			(width 0)
-			(type default)
-		)
-	)
-	(wire
-		(pts
-			(xy 82.55 35.56) (xy 96.52 35.56)
-		)
-		(stroke
-			(width 0)
-			(type default)
-		)
-	)
-	(wire
-		(pts
 			(xy 133.35 132.08) (xy 31.75 132.08)
 		)
@@
 	(wire
 		(pts
+			(xy 39.37 82.55) (xy 135.89 82.55)
+		)
+		(stroke
+			(width 0)
+			(type default)
+		)
+	)
+	(wire
+		(pts
 			(xy 101.6 -3.81) (xy 101.6 -1.27)
 		)
@@
 	(wire
 		(pts
+			(xy 39.37 77.47) (xy 139.7 77.47)
+		)
+		(stroke
+			(width 0)
+			(type default)
+		)
+	)
+	(wire
+		(pts
 			(xy 91.44 -1.27) (xy 91.44 17.78)
 		)
@@
 	(wire
 		(pts
+			(xy 139.7 20.32) (xy 139.7 77.47)
+		)
+		(stroke
+			(width 0)
+			(type default)
+		)
+	)
+	(wire
+		(pts
 			(xy 118.11 1.27) (xy 135.89 1.27)
 		)
@@
 	(wire
 		(pts
+			(xy 91.44 73.66) (xy 91.44 17.78)
+		)
+		(stroke
+			(width 0)
+			(type default)
+		)
+	)
+	(wire
+		(pts
 			(xy 82.55 30.48) (xy 96.52 30.48)
 		)
@@
 		(pts
 			(xy 91.44 17.78) (xy 96.52 17.78)
+		)
+		(stroke
+			(width 0)
+			(type default)
+		)
+	)
+	(wire
+		(pts
+			(xy 135.89 17.78) (xy 135.89 82.55)
 		)
 		(stroke
@@
 	(sheet
 		(at 13.335 60.96)
-		(size 26.67 36.83)
+		(size 26.035 36.83)
 		(exclude_from_sim no)
 		(in_bom yes)
@@
 		)
 		(property "Sheetname" "PORTS"
-			(at 12.6234 97.79 90)
+			(at 13.335 60.2484 0)
 			(effects
 				(font
@@
 		)
 		(property "Sheetfile" "PORTS.kicad_sch"
-			(at 40.5896 97.79 90)
+			(at 13.335 98.3746 0)
 			(effects
 				(font
@@
 			(effects
 				(font
+					(size 1.27 1.27)
+				)
+				(justify right)
+			)
+		)
+		(pin "GPIO_26" input
+			(at 39.37 73.66 0)
+			(effects
+				(font
+					(size 1.27 1.27)
+				)
+				(justify right)
+			)
+		)
+		(pin "GPIO_27" input
+			(at 39.37 77.47 0)
+			(effects
+				(font
+					(size 1.27 1.27)
+				)
+				(justify right)
+			)
+		)
+		(pin "GPIO_28" input
+			(at 39.37 82.55 0)
+			(effects
+				(font

Commit message: Updated PCB files
Other:
- sheet MCU (page 4) ports: added none; removed GPIO_20
- sheet Relays+RC SNUBBER ports: added none; removed GPIO_20
Changed lines of the file:
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@@
-	(wire
-		(pts
-			(xy 82.55 30.48) (xy 96.52 30.48)
-		)
-		(stroke
-			(width 0)
-			(type default)
-		)
-	)
 	(wire
 		(pts
@@
 			)
 		)
-		(pin "GPIO_20" output
-			(at 82.55 30.48 0)
-			(effects
-				(font
-					(size 1.27 1.27)
-				)
-				(justify right)
-			)
-		)
 		(pin "L_FUSED" output
 			(at 53.34 33.02 180)
@@
 			(effects
 				(font
-					(size 1.27 1.27)
-				)
-				(justify left)
-			)
-		)
-		(pin "GPIO_20" output
-			(at 96.52 30.48 180)
-			(effects
-				(font
