File: MCU.kicad_sch (KiCad schematic)
At the start: 7 parts, among them U2 RaspberryPi_Pico

Commit message: SCHEMATIC CONTINUATION
Parts:
- removed C10: 10u, Capacitor_SMD:C_0603_1608Metric, symbol Device:C
- renumbered C9 to C10, C8 to C11, R1 to R15
Connections:
- net 3V3: now reaches C11.1, U2.36 (3V3)
- net GPIO_13: now reaches U2.17 (GPIO13)
- net GPIO_14: now reaches U2.19 (GPIO14)
Changed lines of the file:
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@@
+	(wire
+		(pts
+			(xy 114.3 106.68) (xy 120.65 106.68)
+		)
+		(stroke
+			(width 0)
+			(type default)
+		)
+	)
 	(wire
 		(pts
@@
 		(pts
 			(xy 52.07 63.5) (xy 52.07 71.12)
+		)
+		(stroke
+			(width 0)
+			(type default)
+		)
+	)
+	(wire
+		(pts
+			(xy 114.3 109.22) (xy 120.65 109.22)
 		)
 		(stroke
@@
 		)
 	)
+	(global_label "3V3"
+		(shape input)
+		(at 148.59 41.91 90)
+		(fields_autoplaced yes)
+		(effects
+			(font
+				(size 1.27 1.27)
+				(thickness 0.254)
+				(bold yes)
+			)
+			(justify left)
+		)
+		(property "Intersheetrefs" "${INTERSHEET_REFS}"
+			(at 148.59 34.9412 90)
+			(effects
+				(font
+					(size 1.27 1.27)
+				)
+				(justify left)
+				(hide yes)
+			)
+		)
+	)
 	(hierarchical_label "GPIO_20"
 		(shape output)
@@
 		)
 	)
+	(hierarchical_label "GPIO_13"
+		(shape input)
+		(at 114.3 106.68 180)
+		(effects
+			(font
+				(size 1.27 1.27)
+			)
+			(justify right)
+		)
+	)
 	(hierarchical_label "GPIO_11"
 		(shape output)
@@
 				(thickness 0.254)
 				(bold yes)
+			)
+			(justify right)
+		)
+	)
+	(hierarchical_label "GPIO_14"
+		(shape input)
+		(at 114.3 109.22 180)
+		(effects
+			(font
+				(size 1.27 1.27)
 			)
 			(justify right)
@@
 		(dnp no)
 		(fields_autoplaced yes)
-		(property "Reference" "#PWR018"
+		(property "Reference" "#PWR017"
 			(at 143.51 144.78 0)
 			(effects
@@
 			(project "ECM Synchronika Custom Control Board"
 				(path "/0a1cfe74-4adf-4cda-8eff-54fb631bdb34/fa757c9b-92b6-48f7-b60b-b85d2ef688f7"
-					(reference "#PWR018")
+					(reference "#PWR017")
 					(unit 1)
 				)
@@
 		(dnp no)
 		(fields_autoplaced yes)
-		(property "Reference" "C8"
+		(property "Reference" "C11"
 			(at 161.29 34.29 90)
 			(effects
@@
 			(project "ECM Synchronika Custom Control Board"
 				(path "/0a1cfe74-4adf-4cda-8eff-54fb631bdb34/fa757c9b-92b6-48f7-b60b-b85d2ef688f7"
-					(reference "C8")
+					(reference "C11")
 					(unit 1)
 				)
@@
 		(dnp no)
 		(fields_autoplaced yes)
-		(property "Reference" "#PWR017"
+		(property "Reference" "#PWR016"
 			(at 116.84 50.8 0)
 			(effects
@@
 			(project "ECM Synchronika Custom Control Board"
 				(path "/0a1cfe74-4adf-4cda-8eff-54fb631bdb34/fa757c9b-92b6-48f7-b60b-b85d2ef688f7"
-					(reference "#PWR017")
+					(reference "#PWR016")
 					(unit 1)
 				)
@@
 		(dnp no)
 		(fields_autoplaced yes)
-		(property "Reference" "R1"
+		(property "Reference" "R15"
 			(at 54.61 76.1999 0)
 			(effects
@@
 			(project "ECM Synchronika Custom Control Board"
 				(path "/0a1cfe74-4adf-4cda-8eff-54fb631bdb34/fa757c9b-92b6-48f7-b60b-b85d2ef688f7"
-					(reference "R1")
+					(reference "R15")
 					(unit 1)
 				)
@@
 		(dnp no)
 		(fields_autoplaced yes)
-		(property "Reference" "#PWR016"
+		(property "Reference" "#PWR018"
 			(at 167.64 50.8 0)
 			(effects
@@
 			(project "ECM Synchronika Custom Control Board"
 				(path "/0a1cfe74-4adf-4cda-8eff-54fb631bdb34/fa757c9b-92b6-48f7-b60b-b85d2ef688f7"
-					(reference "#PWR016")
+					(reference "#PWR018")
 					(unit 1)
 				)
@@
 	(symbol
 		(lib_id "Device:C")
-		(at 116.84 19.05 0)
-		(unit 1)
-		(exclude_from_sim no)
-		(in_bom yes)
-		(on_board yes)
-		(dnp no)
-		(fields_autoplaced yes)
-		(property "Reference" "C10"
-			(at 120.65 17.7799 0)
-			(effects
-				(font
-					(size 1.27 1.27)
-				)
-				(justify left)
-			)
-		)
-		(property "Value" "10u"
-			(at 120.65 20.3199 0)
-			(effects
-				(font
-					(size 1.27 1.27)
-				)
-				(justify left)
-			)
-		)
-		(property "Footprint" "Capacitor_SMD:C_0603_1608Metric"
-			(at 117.8052 22.86 0)
-			(effects
-				(font
-					(size 1.27 1.27)
-				)
-				(hide yes)
-			)
-		)
-		(property "Datasheet" "~"
-			(at 116.84 19.05 0)
-			(effects
-				(font
-					(size 1.27 1.27)
-				)
-				(hide yes)
-			)
-		)
-		(property "Description" "Unpolarized capacitor"
-			(at 116.84 19.05 0)
-			(effects
-				(font
-					(size 1.27 1.27)
-				)
-				(hide yes)
-			)
-		)
-		(pin "1"
-		)
-		(pin "2"
-		)
-		(instances
-			(project "ECM Synchronika Custom Control Board"
-				(path "/0a1cfe74-4adf-4cda-8eff-54fb631bdb34/fa757c9b-92b6-48f7-b60b-b85d2ef688f7"
-					(reference "C10")
-					(unit 1)
-				)
-			)
-		)
-	)
-	(symbol
-		(lib_id "Device:C")
 		(at 123.19 39.37 90)
 		(unit 1)
@@
 		(dnp no)
 		(fields_autoplaced yes)
-		(property "Reference" "C9"
+		(property "Reference" "C10"
 			(at 123.19 31.75 90)
 			(effects
@@
 			(project "ECM Synchronika Custom Control Board"
 				(path "/0a1cfe74-4adf-4cda-8eff-54fb631bdb34/fa757c9b-92b6-48f7-b60b-b85d2ef688f7"
-					(reference "C9")
+					(reference "C10")
 					(unit 1)
 				)

Commit message: Update KiCad project files
Parts:
- added BZ1: Buzzer, Buzzer_Beeper:Buzzer_12x9.5RM7.6, symbol Device:Buzzer
- added D16: LED, LED_SMD:LED_0805_2012Metric, symbol Device:LED
- added R48, R49: 330, Resistor_SMD:R_0805_2012Metric, symbol Device:R
Connections:
- net GND: now also BZ1.2 (-), D16.2 (A)
- net GPIO0: now reaches U2.1 (GPIO0)
- net GPIO7: now reaches U2.10 (GPIO7)
- net GPIO8: now reaches U2.11 (GPIO8)
- net GPIO9: now reaches U2.12 (GPIO9)
- net GPIO1: now reaches U2.2 (GPIO1)
- net at U2.20 (GPIO15): now also R48.1
- net GPIO_16: now reaches U2.21 (GPIO16)
- net GPIO_17: now reaches U2.22 (GPIO17)
- net GPIO_18: now reaches U2.24 (GPIO18)
- net at U2.25 (GPIO19): now also R49.1
- net GPIO21: now reaches U2.27 (GPIO21)
- net GPIO22: now reaches U2.29 (GPIO22)
- net GPIO_2: now reaches U2.4 (GPIO2)
- net GPIO_3: now reaches U2.5 (GPIO3)
- net GPIO_5: now reaches U2.7 (GPIO5)
- net GPIO6: now reaches U2.9 (GPIO6)
- new net: BZ1.1 (+), R49.2
- new net: D16.1 (K), R48.2
- no-connect marks 0 -> 1

Commit message: Update KiCad project files
Parts:
- removed U2: RaspberryPi_Pico, Module:RaspberryPi_Pico_Common_Unspecified, symbol MCU_Module:RaspberryPi_Pico
- added A1: RaspberryPi_Pico, Module:RaspberryPi_Pico_SMD, symbol MCU_Module:RaspberryPi_Pico_Extensive
- added S2: EVQ-P7A01P, EVQ-P7A01P:SW_EVQ-P7A01P, symbol SMD SWITCH:EVQ-P7A01P
Connections:
- net +5v: now also A1.39 (VSYS)
- net 3V3: now also A1.36 (3V3)
- net 3V3-EN: now also A1.37 (3V3_EN)
- net ADC-REF: now also A1.35 (ADC_VREF)
- net GND: now also S1.1_1, S1.1_2, A1.13 (GND), A1.18 (GND), A1.23 (GND), A1.28 (GND), A1.3 (GND), A1.38 (GND), A1.8 (GND), A1.D2 (GND), S2.1_1, S2.1_2
- net GNDA: now also A1.33 (AGND)
- net GPIO0: now also A1.1 (GPIO0)
- net GPIO1: now also A1.2 (GPIO1)
- net GPIO21: now also A1.27 (GPIO21)
- net GPIO22: now also A1.29 (GPIO22)
- net GPIO6: now also A1.9 (GPIO6)
- net GPIO7: now also A1.10 (GPIO7)
- net GPIO8: now also A1.11 (GPIO8)
- net GPIO9: now also A1.12 (GPIO9)
- net GPIO_10: now also A1.14 (GPIO10)
- net GPIO_11: now also A1.15 (GPIO11)
- net GPIO_12: now also A1.16 (GPIO12)
- net GPIO_13: now also A1.17 (GPIO13)
- net GPIO_14: now also A1.19 (GPIO14)
- net GPIO_16: now also A1.21 (GPIO16)
- net GPIO_17: now also A1.22 (GPIO17)
- net GPIO_18: now also A1.24 (GPIO18)
- net GPIO_2: now also A1.4 (GPIO2)
- net GPIO_20: now also A1.26 (GPIO20)
- net GPIO_3: now also A1.5 (GPIO3)
- net GPIO_5: now also A1.7 (GPIO5)
- net at R48.1: now also A1.20 (GPIO15)
- net at R49.1: now also A1.25 (GPIO19)
- net PIN_RUN: now reaches R15.2, S1.2_1, S1.2_2
- net PIN_RUN: now also A1.30 (RUN)
- new net B00T_SEL: A1.TP6 (~{BOOTSEL}), S2.2_1, S2.2_2
- new net GPIO_26: A1.31 (GPIO26_ADC0)
- new net GPIO_27: A1.32 (GPIO27_ADC1)
- new net GPIO_28: A1.34 (GPIO28_ADC2)
- new net GPIO_4: A1.6 (GPIO4)
- no-connect marks 1 -> 7
Other:
- moved on the sheet: D16, R48

Commit message: Update KiCad project files
Parts:
- removed S1, S2: EVQ-P7A01P, EVQ-P7A01P:SW_EVQ-P7A01P, symbol SMD SWITCH:EVQ-P7A01P
- added SW1, SW2: SW_Push, Button_Switch_THT:SW_PUSH_6mm, symbol Switch:SW_Push
Connections:
- net 3V3 is gone; now on net +3V3: A1.36 (3V3), C11.1
- net B00T_SEL: now also SW2.2
- net GND: now also SW1.1, SW2.1
- net PIN_RUN: now also SW1.2
Other:
- note added: "BOOT_BOTTON"
- note added: "RESET_BUTTON"
- note removed: "RESER_BUTTON"

Commit message: Updated PCB files
Connections:
- net GPIO_20: no longer names the net of A1.26 (GPIO20)
- no-connect marks 7 -> 8
Changed lines of the file:
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@@
+	)
+	(no_connect
+		(at 173.99 86.36)
 	)
 	(no_connect
@@
 		(effects
 			(font
-				(size 1.27 1.27)
-				(thickness 0.254)
-				(bold yes)
-			)
-			(justify left)
-		)
-	)
-	(hierarchical_label "GPIO_20"
-		(shape output)
-		(at 173.99 86.36 0)
-		(effects
-			(font
