File: ECM Synchronika Custom Control Board.kicad_pcb (KiCad board)
At the start: 2 copper layers, 17 parts, among them J1 Screw_Terminal_01x03, U1 AP2112K-3.3

Commit message: Update KiCad project files
Parts:
- removed A1: RaspberryPi_Pico, Module:RaspberryPi_Pico_Common_Unspecified
- added C11: 100n, Capacitor_SMD:C_0603_1608Metric, F.Cu at (78.4, 87.6)
- added C12: 100n, Capacitor_SMD:C_0805_2012Metric, F.Cu at (58.9, 162.5)
- added C13: 100n, Capacitor_SMD:C_0805_2012Metric, F.Cu at (58.9, 165.5)
- added C14: 10n, Capacitor_SMD:C_0805_2012Metric, F.Cu at (58.9, 168.5)
- added C15: 100n, Capacitor_SMD:C_0805_2012Metric, F.Cu at (58.9, 171.6)
- added C16: 100n, Capacitor_SMD:C_0805_2012Metric, F.Cu at (58.9, 174.6)
- added D1: 1N4007, Diode_THT:D_DO-41_SOD81_P10.16mm_Horizontal, F.Cu at (120.2, 116.4)
- added D10: LED, LED_SMD:LED_0805_2012Metric, F.Cu at (149.8, 158.9)
- added D11: PESD5V0S1UL, Diode_SMD:D_SOD-882, F.Cu at (78.7, 168.8)
- added D12: PESD5V0S1UL, Diode_SMD:D_SOD-882, F.Cu at (78.7, 171.1)
- added D2: 1N4007, Diode_THT:D_DO-41_SOD81_P10.16mm_Horizontal, F.Cu at (120.2, 120.6)
- added D3: LED, LED_SMD:LED_0805_2012Metric, F.Cu at (134.5, 115.8)
- added D4: LED, LED_SMD:LED_0805_2012Metric, F.Cu at (134.5, 118.8)
- added D5: 1N4007, Diode_THT:D_DO-41_SOD81_P10.16mm_Horizontal, F.Cu at (120.2, 124.9)
- added D6: LED, LED_SMD:LED_0805_2012Metric, F.Cu at (134.5, 121.9)
- added D7: 1N4007, Diode_THT:D_DO-41_SOD81_P10.16mm_Horizontal, F.Cu at (120.2, 129.1)
- added D8: LED, LED_SMD:LED_0805_2012Metric, F.Cu at (134.5, 124.9)
- added D9: LED, LED_SMD:LED_0805_2012Metric, F.Cu at (149.8, 155.8)
- added J10: 928814-1, 6.3mm spade:TE_928814-1, F.Cu at (150.2, 127.8)
- added J11: 928814-1, 6.3mm spade:TE_928814-1, F.Cu at (150.2, 122.5)
- added J12: 928814-1, 6.3mm spade:TE_928814-1, F.Cu at (150.2, 117.2)
- added J13: 928814-1, 6.3mm spade:TE_928814-1, F.Cu at (150.2, 112.0)
- added J14: 928814-1, 6.3mm spade:TE_928814-1, F.Cu at (150.2, 106.7)
- added J15: 928814-1, 6.3mm spade:TE_928814-1, F.Cu at (150.2, 101.4)
- added J2: Screw_Terminal_01x02, TerminalBlock_Phoenix:TerminalBlock_Phoenix_MKDS-1-2-3.81_1x02_P3.81mm_Horizontal, F.Cu at (136.4, 149.8)
- added J3: Screw_Terminal_01x02, TerminalBlock_Phoenix:TerminalBlock_Phoenix_MKDS-1-2-3.81_1x02_P3.81mm_Horizontal, F.Cu at (136.4, 159.4)
- added J4: Screw_Terminal_01x02, TerminalBlock_Phoenix:TerminalBlock_Phoenix_MKDS-1,5-2-5.08_1x02_P5.08mm_Horizontal, F.Cu at (64.7, 167.3)
- added J5: Screw_Terminal_01x03, TerminalBlock_Phoenix:TerminalBlock_Phoenix_MKDS-1,5-3-5.08_1x03_P5.08mm_Horizontal, F.Cu at (64.7, 179.4)
- added J6: 928814-1, 6.3mm spade:TE_928814-1, F.Cu at (150.2, 90.5)
- added J7: 928814-1, 6.3mm spade:TE_928814-1, F.Cu at (150.4, 84.3)
- added J8: 928814-1, 6.3mm spade:TE_928814-1, F.Cu at (150.2, 138.4)
- added J9: 928814-1, 6.3mm spade:TE_928814-1, F.Cu at (150.2, 133.1)
- added K1: G2RL-1-H, Relay_THT:Relay_SPDT_Omron_G2RL-1, F.Cu at (88.8, 87.0)
- added K2: G2RL-1-H, Relay_THT:Relay_SPDT_Omron_G2RL-1, F.Cu at (103.0, 87.0)
- added K3: G2RL-1-H, Relay_THT:Relay_SPDT_Omron_G2RL-1, F.Cu at (117.1, 87.0)
- added K4: G2RL-1-H, Relay_THT:Relay_SPDT_Omron_G2RL-1, F.Cu at (131.3, 87.0)
- added NT1: NetTie_2, NetTie:NetTie-2_SMD_Pad2.0mm, F.Cu at (79.9, 92.8)
- added Q1: MMBT2222A, Package_TO_SOT_SMD:SOT-23, F.Cu at (115.9, 116.7)
- added Q2: MMBT2222A, Package_TO_SOT_SMD:SOT-23, F.Cu at (115.9, 121.3)
- added Q3: MMBT2222A, Package_TO_SOT_SMD:SOT-23, F.Cu at (115.9, 125.9)
- added Q4: MMBT2222A, Package_TO_SOT_SMD:SOT-23, F.Cu at (115.9, 130.5)
- added Q5: MMBT2222A, Package_TO_SOT_SMD:SOT-23, F.Cu at (150.0, 147.5)
- added Q6: MMBT2222A, Package_TO_SOT_SMD:SOT-23, F.Cu at (150.0, 152.1)
- added R1: 1K, Resistor_SMD:R_0805_2012Metric, F.Cu at (120.6, 132.7)
- added R10: 1K, Resistor_SMD:R_0805_2012Metric, F.Cu at (129.4, 132.7)
- added R11: 470, Resistor_SMD:R_0805_2012Metric, F.Cu at (129.4, 135.7)
- added R12: 10K, Resistor_SMD:R_0805_2012Metric, F.Cu at (129.4, 138.6)
- added R13: 10K, Resistor_SMD:R_0805_2012Metric, F.Cu at (129.4, 141.6)
- added R14: 100, Resistor_SMD:R_1210_3225Metric, F.Cu at (134.4, 137.6)
- added R15: 10K, Resistor_SMD:R_0603_1608Metric, F.Cu at (78.4, 90.1)
- added R16: 1K, Resistor_SMD:R_0805_2012Metric, F.Cu at (145.3, 146.5)
- added R17: 10K, Resistor_SMD:R_0805_2012Metric, F.Cu at (145.3, 149.5)
- added R18: 1K, Resistor_SMD:R_0805_2012Metric, F.Cu at (145.3, 152.4)
- added R19: 1K, Resistor_SMD:R_0805_2012Metric, F.Cu at (145.3, 155.4)
- added R2: 1K, Resistor_SMD:R_0805_2012Metric, F.Cu at (120.6, 135.7)
- added R20: 10K, Resistor_SMD:R_0805_2012Metric, F.Cu at (145.3, 158.3)
- added R21: 1K, Resistor_SMD:R_0805_2012Metric, F.Cu at (145.3, 161.3)
- added R22: 1K, Resistor_SMD:R_0805_2012Metric, F.Cu at (54.5, 162.5)
- added R23: 3.3K, Resistor_SMD:R_0805_2012Metric, F.Cu at (54.5, 165.4)
- added R24: 1.2K, Resistor_SMD:R_0805_2012Metric, F.Cu at (54.5, 168.4)
- added R25: 1K, Resistor_SMD:R_0805_2012Metric, F.Cu at (54.5, 171.3)
- added R26: 4.7K, Resistor_SMD:R_0805_2012Metric, F.Cu at (54.5, 174.3)
- added R27: 10K, Resistor_SMD:R_0805_2012Metric, F.Cu at (54.5, 177.2)
- added R3: 470, Resistor_SMD:R_0805_2012Metric, F.Cu at (120.6, 138.6)
- added R4: 470, Resistor_SMD:R_0805_2012Metric, F.Cu at (120.6, 141.6)
- added R5: 10K, Resistor_SMD:R_0805_2012Metric, F.Cu at (125.0, 132.7)
- added R6: 10K, Resistor_SMD:R_0805_2012Metric, F.Cu at (125.0, 135.7)
- added R7: 100, Resistor_SMD:R_1210_3225Metric, F.Cu at (134.4, 133.4)
- added R8: 1K, Resistor_SMD:R_0805_2012Metric, F.Cu at (125.0, 138.6)
- added R9: 470, Resistor_SMD:R_0805_2012Metric, F.Cu at (125.0, 141.6)
- added TH1: 50k NTC, Resistor_SMD:R_0603_1608Metric, F.Cu at (75.3, 168.9)
- added TH2: 50k NTC, Resistor_SMD:R_0603_1608Metric, F.Cu at (75.3, 171.4)
- added U2: RaspberryPi_Pico, Module:RaspberryPi_Pico_Common_Unspecified, F.Cu at (64.3, 131.9)
- added U3: MAX31855KASA, Package_SO:SOIC-8_3.9x4.9mm_P1.27mm, F.Cu at (77.6, 164.4)
- C1: footprint Capacitor_THT:C_Rect_L18.0mm_W9.0mm_P15.00mm_FKS3_FKP3 -> Capacitor_THT:C_Rect_L18.0mm_W5.0mm_P15.00mm_FKS3_FKP3
- C10: value 10u -> 100n
- C2: value C -> 100u; footprint Capacitor_THT:C_Radial_D6.3mm_H7.0mm_P2.50mm -> Capacitor_SMD:CP_Elec_6.3x5.9
- C3: value 100u -> 100n; footprint Capacitor_THT:C_Radial_D6.3mm_H7.0mm_P2.50mm -> Capacitor_THT:C_Rect_L26.5mm_W11.5mm_P22.50mm_MKS4
- C4: value 47u -> 100n; footprint Capacitor_SMD:C_1206_3216Metric -> Capacitor_THT:C_Rect_L26.5mm_W11.5mm_P22.50mm_MKS4
- C5: value 100n -> 100u; footprint Capacitor_SMD:C_0805_2012Metric -> Capacitor_SMD:CP_Elec_6.3x5.9
- C6: value 100n -> 47u; footprint Capacitor_SMD:C_0805_2012Metric -> Capacitor_SMD:C_1206_3216Metric
- C7: value 22U -> 100n; footprint Capacitor_SMD:C_1206_3216Metric -> Capacitor_SMD:C_0805_2012Metric
- C8: value 100n -> 22U; footprint Capacitor_SMD:C_0603_1608Metric -> Capacitor_SMD:C_1206_3216Metric
- C9: footprint Capacitor_SMD:C_0603_1608Metric -> Capacitor_SMD:C_0805_2012Metric
- F1: value Fuse -> Fuse_Small; footprint Fuse:Fuseholder_Clip-5x20mm_Littelfuse_100_Inline_P20.50x4.60mm_D1.30mm_Horizontal -> Fuse:Fuseholder_Clip-5x20mm_Littelfuse_111_Inline_P20.00x5.00mm_D1.05mm_Horizontal
- J1: value Screw_Terminal_01x03 -> 928814-1; footprint TerminalBlock_MetzConnect:TerminalBlock_MetzConnect_Type701_RT11L03HGLU_1x03_P6.35mm_Horizontal -> 6.3mm spade:TE_928814-1
- PS1: footprint HLK-5M05:CONV_HLK-5M05 -> HLK_5M05:CONV_HLK-5M05
- RV1: footprint Varistor:RV_Disc_D15.5mm_W5mm_P7.5mm -> Varistor:RV_Disc_D15.5mm_W4.9mm_P7.5mm
- moved PS1 139.2 mm to (103.2, 156.6)
- moved F1 130.9 mm to (103.0, 173.0)
- moved C1 114.4 mm to (103.5, 179.7)
- moved RV1 112.5 mm to (106.0, 185.1)
- moved C8 96.1 mm to (136.3, 179.5)
- moved C2 94.9 mm to (126.1, 180.5)
- moved C6 91.2 mm to (136.3, 176.1)
- moved U1 88.6 mm to (142.3, 179.9)
- moved C5 88.0 mm to (138.8, 170.4)
- moved C9 84.5 mm to (146.3, 170.8)
- moved FB1 84.3 mm to (146.2, 175.7)
- moved C7 80.3 mm to (146.3, 167.8)
- moved C4 79.9 mm to (88.2, 133.8)
- moved C10 67.7 mm to (78.4, 85.1)
- moved C3 57.1 mm to (88.2, 120.8)
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Connections:
- C1 pad 1: unconnected-(C1-Pad1) -> /HV_INPUT + PROTECTION/L_FUSED
- C1 pad 2: unconnected-(C1-Pad2) -> /HV_INPUT + PROTECTION/NEUTRAL
- C10 pad 1: unconnected-(C10-Pad1) -> GND
- C10 pad 2: unconnected-(C10-Pad2) -> +5v
- C2 pad 1: unconnected-(C2-Pad1) -> +5v
- C2 pad 2: unconnected-(C2-Pad2) -> GND
- C3 pad 1: unconnected-(C3-Pad1) -> /Relays+RC SNUBBER/PUMP_LOAD
- C3 pad 2: unconnected-(C3-Pad2) -> Net-(C3-Pad2)
- C4 pad 1: unconnected-(C4-Pad1) -> Net-(C4-Pad1)
- C4 pad 2: unconnected-(C4-Pad2) -> /HV_INPUT + PROTECTION/L_FUSED
- C5 pad 1: unconnected-(C5-Pad1) -> +5v
- C5 pad 2: unconnected-(C5-Pad2) -> GND
- C6 pad 1: unconnected-(C6-Pad1) -> Net-(U1-VOUT)
- C6 pad 2: unconnected-(C6-Pad2) -> GND
- C7 pad 1: unconnected-(C7-Pad1) -> Net-(U1-VOUT)
- C7 pad 2: unconnected-(C7-Pad2) -> GND
- C8 pad 1: unconnected-(C8-Pad1) -> Net-(C8-Pad1)
- C8 pad 2: unconnected-(C8-Pad2) -> GND
- C9 pad 1: unconnected-(C9-Pad1) -> ADC-REF
- C9 pad 2: unconnected-(C9-Pad2) -> GND
- F1 pad 1: unconnected-(F1-Pad1) -> /HV_INPUT + PROTECTION/LIVE
- F1 pad 2: unconnected-(F1-Pad2) -> /HV_INPUT + PROTECTION/L_FUSED
- FB1 pad 1: unconnected-(FB1-Pad1) -> Net-(C8-Pad1)
- FB1 pad 2: unconnected-(FB1-Pad2) -> ADC-REF
- J1 pad 1: unconnected-(J1-Pin_1-Pad1) -> /HV_INPUT + PROTECTION/NEUTRAL
- J1 pad 2: unconnected-(J1-Pin_2-Pad2) -> (no net)
- PS1 pad 1: unconnected-(PS1-AC1-Pad1) -> /HV_INPUT + PROTECTION/L_FUSED
- PS1 pad 2: unconnected-(PS1-AC2-Pad2) -> /HV_INPUT + PROTECTION/NEUTRAL
- PS1 pad 3: unconnected-(PS1--VO-Pad3) -> GND
- PS1 pad 4: unconnected-(PS1-+VO-Pad4) -> +5v
- RV1 pad 1: unconnected-(RV1-Pad1) -> /HV_INPUT + PROTECTION/LIVE
- RV1 pad 2: unconnected-(RV1-Pad2) -> /HV_INPUT + PROTECTION/NEUTRAL
- U1 pad 1: unconnected-(U1-VIN-Pad1) -> +5v
- U1 pad 2: unconnected-(U1-GND-Pad2) -> GND
- U1 pad 3: unconnected-(U1-EN-Pad3) -> 3V3-EN
- U1 pad 5: unconnected-(U1-VOUT-Pad5) -> Net-(U1-VOUT)
Other:
- board outline added: 119.4 x 113.1 mm

Commit message: Update KiCad project files
Parts:
- removed J13: 928814-1, 6.3mm spade:TE_928814-1
- removed U2: RaspberryPi_Pico, Module:RaspberryPi_Pico_Common_Unspecified
- added A1: RaspberryPi_Pico, Module:RaspberryPi_Pico_SMD, F.Cu at (182.6, 90.4)
- added BZ1: Buzzer, Buzzer_Beeper:Buzzer_12x9.5RM7.6, F.Cu at (188.8, 60.9)
- added C17: 100n, Capacitor_SMD:C_0603_1608Metric, B.Cu at (181.7, 87.6)
- added C18: 100n, Capacitor_SMD:C_0603_1608Metric, B.Cu at (183.7, 71.5)
- added C19: 100n, Capacitor_SMD:C_0603_1608Metric, B.Cu at (183.7, 69.9)
- added C20: 1u, Capacitor_SMD:C_0603_1608Metric, B.Cu at (184.0, 73.2)
- added C21: 100n, Capacitor_SMD:C_0603_1608Metric, B.Cu at (184.0, 75.8)
- added C22: 100n, Capacitor_SMD:C_0603_1608Metric, B.Cu at (181.7, 90.7)
- added C23: C_Polarized, Capacitor_SMD:CP_Elec_5x5.4, F.Cu at (159.6, 56.3)
- added C24: 100u, Capacitor_SMD:CP_Elec_6.3x5.9, F.Cu at (153.5, 106.1)
- added D13: PESD5V0S1UL, Diode_SMD:D_SOD-882, F.Cu at (179.0, 48.5)
- added D14: PESD5V0S1UL, Diode_SMD:D_SOD-882, F.Cu at (175.8, 48.6)
- added D15: PESD5V0S1UL, Diode_SMD:D_SOD-882, F.Cu at (168.6, 48.8)
- added D16: LED, LED_SMD:LED_0805_2012Metric, F.Cu at (254.0, 70.2)
- added D17: SMBJ5.0A, D(5V):DIOM4336X265N, F.Cu at (151.6, 86.9)
- added FB2: FerriteBead, Inductor_SMD:L_0603_1608Metric, F.Cu at (148.4, 104.6)
- added H1: MountingHole_Pad, MountingHole:MountingHole_3.2mm_M3_ISO7380_Pad_TopBottom, F.Cu at (83.0, 45.3)
- added H2: MountingHole, MountingHole:MountingHole_3.2mm_M3_ISO14580, F.Cu at (203.5, 44.8)
- added H3: MountingHole, MountingHole:MountingHole_3.2mm_M3_ISO14580, F.Cu at (201.5, 111.4)
- added H4: MountingHole, MountingHole:MountingHole_3.2mm_M3_ISO14580, F.Cu at (83.0, 108.8)
- added J16: 928814-1, 6.3mm spade:TE_928814-1, F.Cu at (182.5, 44.9)
- added J17: 928814-1, 6.3mm spade:TE_928814-1, F.Cu at (179.0, 44.8)
- added J18: 928814-1, 6.3mm spade:TE_928814-1, F.Cu at (175.6, 44.8)
- added J19: 928814-1, 6.3mm spade:TE_928814-1, F.Cu at (172.1, 44.8)
- added J20: 928814-1, 6.3mm spade:TE_928814-1, F.Cu at (168.6, 44.8)
- added J21: 928814-1, 6.3mm spade:TE_928814-1, F.Cu at (164.8, 44.9)
- added J22: 928814-1, 6.3mm spade:TE_928814-1, F.Cu at (160.9, 44.9)
- added J23: MTLW-104-X-X-S-X, 4 PIN:SAMTEC_MTLW-104-X-X-S-X, F.Cu at (164.2, 82.2)
- added J24: MTLW-104-X-X-S-X, 4 PIN:SAMTEC_MTLW-104-X-X-S-X, F.Cu at (196.4, 109.5)
- added J25: MTLW-104-X-X-S-X, 4 PIN:SAMTEC_MTLW-104-X-X-S-X, F.Cu at (126.6, 111.7)
- added J26: TSW-105-05-L-S-LL, 5 PIN:SAMTEC_TSW-105-05-L-S-LL, F.Cu at (196.3, 93.7)
- added J27: Screw_Terminal_01x02, TerminalBlock_Phoenix:TerminalBlock_Phoenix_MKDS-1,5-2-5.08_1x02_P5.08mm_Horizontal, F.Cu at (165.3, 110.4)
- added P1: BM08B-GHS-TBT_LF__SN__N_, 8 PIN HEADER:JST_BM08B-GHS-TBT_LF__SN__N_, B.Cu at (204.8, 101.3)
- added R28: 10K, Resistor_SMD:R_0805_2012Metric, B.Cu at (183.8, 68.1)
- added R29: 10K, Resistor_SMD:R_0805_2012Metric, B.Cu at (188.4, 69.3)
- added R30: 10K, Resistor_SMD:R_0805_2012Metric, B.Cu at (188.5, 72.2)
- added R31: 10K, Resistor_SMD:R_0805_2012Metric, B.Cu at (188.1, 74.4)
- added R32: 10K, Resistor_SMD:R_0805_2012Metric, B.Cu at (179.2, 82.7)
- added R33: 10K, Resistor_SMD:R_0805_2012Metric, B.Cu at (182.7, 82.6)
- added R34: 100, Resistor_SMD:R_0805_2012Metric, B.Cu at (179.4, 68.9)
- added R35: 10K, Resistor_SMD:R_0805_2012Metric, B.Cu at (179.4, 71.0)
- added R36: 100K, Resistor_SMD:R_0805_2012Metric, B.Cu at (187.4, 78.3)
- added R37: 100K, Resistor_SMD:R_0805_2012Metric, B.Cu at (179.4, 76.9)
- added R38: 1M, Resistor_SMD:R_0805_2012Metric, B.Cu at (179.4, 79.9)
- added R39: 33, Resistor_SMD:R_0805_2012Metric, B.Cu at (186.7, 97.1)
- added R40: 33, Resistor_SMD:R_0805_2012Metric, B.Cu at (188.4, 106.1)
- added R41: 10K, Resistor_SMD:R_0603_1608Metric, B.Cu at (178.5, 89.2)
- added R42: 10K, Resistor_SMD:R_0603_1608Metric, B.Cu at (188.4, 102.2)
- added R43: 10K, Resistor_SMD:R_0603_1608Metric, B.Cu at (181.7, 85.9)
- added R44: 33, Resistor_SMD:R_0805_2012Metric, B.Cu at (188.4, 109.0)
- added R45: 33, Resistor_SMD:R_0805_2012Metric, B.Cu at (183.2, 97.1)
- added R46: 4.7k, Resistor_SMD:R_0603_1608Metric, B.Cu at (177.6, 104.4)
- added R47: 4.7k, Resistor_SMD:R_0603_1608Metric, B.Cu at (181.7, 89.2)
- added R48: 330, Resistor_SMD:R_0805_2012Metric, F.Cu at (237.0, 66.1)
- added R49: 330, Resistor_SMD:R_0805_2012Metric, F.Cu at (239.4, 70.2)
- added SW1: SW_Push, Button_Switch_THT:SW_PUSH_6mm, F.Cu at (164.4, 59.8)
- added SW2: SW_Push, Button_Switch_THT:SW_PUSH_6mm, F.Cu at (172.9, 59.8)
- added TP1: TestPoint_Alt, Connector_Pin:Pin_D1.0mm_L10.0mm_LooseFit, F.Cu at (159.4, 100.6)
- added TP2: TestPoint_Alt, Connector_Pin:Pin_D1.0mm_L10.0mm_LooseFit, F.Cu at (163.1, 103.2)
- added TP3: TestPoint_Alt, Connector_Pin:Pin_D1.0mm_L10.0mm_LooseFit, F.Cu at (248.6, 92.7)
- added TP4: TestPoint_Alt, Connector_Pin:Pin_D1.0mm_L10.0mm_LooseFit, F.Cu at (157.9, 73.7)
- added TP5: TestPoint_Alt, Connector_Pin:Pin_D1.0mm_L10.0mm_LooseFit, F.Cu at (253.0, 83.8)
- added TP6: TestPoint_Alt, Connector_Pin:Pin_D1.0mm_L10.0mm_LooseFit, F.Cu at (253.0, 88.3)
- added TP7: TestPoint_Alt, Connector_Pin:Pin_D1.0mm_L10.0mm_LooseFit, F.Cu at (158.4, 86.5)
- added U4: OPA342UA, OPA342UA:D8, B.Cu at (187.7, 84.7)
- added U5: TLV3201AIDBVR, COMPARATOR:COMPARTOR_SOT95P280X145-5N, B.Cu at (184.0, 78.3)
- C16, D10, D3, D4, D6, D8, D9, Q1, Q2, Q3, Q4, Q5, Q6, R1, R10, R11, R12, R13, R14, R16, R17, R18, R19, R2, R20, R21, R26, R27, R3, R4, R5, R6, R7, R8, R9, U1: moved to B.Cu
- D1, D2, D5, D7: footprint Diode_THT:D_DO-41_SOD81_P10.16mm_Horizontal -> Diode_SMD:D_SMA; moved to B.Cu
- J12: value 928814-1 -> Screw_Terminal_01x03; footprint 6.3mm spade:TE_928814-1 -> TerminalBlock_Phoenix:TerminalBlock_Phoenix_MKDS-1,5-3-5.08_1x03_P5.08mm_Horizontal
- J2, J3: footprint TerminalBlock_Phoenix:TerminalBlock_Phoenix_MKDS-1-2-3.81_1x02_P3.81mm_Horizontal -> TerminalBlock_Phoenix:TerminalBlock_Phoenix_MKDS-3-2-5.08_1x02_P5.08mm_Horizontal
- K1, K2, K3, K4: footprint Relay_THT:Relay_SPDT_Omron_G2RL-1 -> RELAY:Relay_SPDT_Omron_G2RL-1 MODIFIED
- PS1: footprint HLK_5M05:CONV_HLK-5M05 -> Converter_ACDC:Converter_ACDC_Hi-Link_HLK-5Mxx
- moved J4 176.5 mm to (203.2, 57.9), turned to 90 degrees
- moved C10 172.4 mm to (249.3, 62.4)
- moved C11 168.9 mm to (245.1, 60.0)
- moved J5 167.1 mm to (206.2, 90.4), turned to 90 degrees
- moved R15 165.3 mm to (242.0, 66.4)
- moved R26 151.3 mm to (182.4, 93.5), turned to 180 degrees
- moved R27 145.9 mm to (177.8, 99.3)
- moved C14 144.0 mm to (161.1, 67.1), turned to 90 degrees
- moved C15 143.5 mm to (161.1, 70.7), turned to -90 degrees
- moved C16 142.5 mm to (177.9, 96.1)
- moved C7 142.3 mm to (238.9, 59.7)
- moved C9 142.3 mm to (238.9, 62.8)
- moved R25 140.1 mm to (168.8, 90.4), turned to -90 degrees
- moved R23 131.8 mm to (169.4, 101.0), turned to 90 degrees
- moved R24 131.5 mm to (169.4, 104.6), turned to -90 degrees
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Connections:
- net /HV_INPUT + PROTECTION/NEUTRAL renamed /HV_INPUT + PROTECTION/N_FUSED
- net /SENSOR INPUT/GPIO_26 renamed /MCU (page 4)/GPIO_26
- net /SENSOR INPUT/GPIO_27 renamed /MCU (page 4)/GPIO_27
- C11 pad 1: 3V3 -> +3V3
- C12 pad 2: GND -> GNDA
- C13 pad 2: GND -> GNDA
- C14 pad 2: GND -> GNDA
- C15 pad 1: GND -> GNDA
- C15 pad 2: 3V3 -> +3V3
- C2 pad 1: +5v -> Net-(PS1-+Vout)
- C6 pad 1: Net-(U1-VOUT) -> +3V3
- C7 pad 1: Net-(U1-VOUT) -> +3V3
- C8 pad 1: Net-(C8-Pad1) -> +3V3
- D10 pad 2: /SSR/SSR_INPUT_- -> Net-(D10-A)
- D11 pad 2: GND -> GNDA
- D12 pad 2: GND -> GNDA
- D9 pad 2: /SSR/SSR_INPUT_- -> Net-(D9-A)
- FB1 pad 1: Net-(C8-Pad1) -> +3V3
- J12 pad 1: /Relays+RC SNUBBER/SPARE_LOAD -> Net-(J12-Pin_1)
- J12 pad 2: (no net) -> /Relays+RC SNUBBER/SPARE_LOAD
- J2 pad 2: /SSR/SSR_INPUT_- -> Net-(D9-A)
- J3 pad 2: /SSR/SSR_INPUT_- -> Net-(D10-A)
- K3 pad 11: /HV_INPUT + PROTECTION/L_FUSED -> Net-(J12-Pin_1)
- K3 pad 12: unconnected-(K3-Pad12) -> Net-(J12-Pin_3)
- PS1 pad 4: +5v -> Net-(PS1-+Vout)
- Q5 pad 3: /SSR/SSR_INPUT_- -> Net-(D9-A)
- Q6 pad 3: /SSR/SSR_INPUT_- -> Net-(D10-A)
- R1 pad 1: /MCU/GPIO_10 -> /MCU (page 4)/GPIO_10
- R10 pad 1: /MCU/GPIO_11 -> /MCU (page 4)/GPIO_11
- R15 pad 2: Net-(R15-Pad2) -> PIN_RUN
- R16 pad 1: /MCU/GPIO_13 -> /MCU (page 4)/GPIO_13
- R19 pad 1: /MCU/GPIO_14 -> /MCU (page 4)/GPIO_14
- R2 pad 1: /MCU/GPIO_12 -> /MCU (page 4)/GPIO_12
- R8 pad 1: /MCU/GPIO_20 -> /MCU (page 4)/GPIO_20
- TH1 pad 2: GND -> GNDA
- TH2 pad 2: GND -> GNDA
- U1 pad 5: Net-(U1-VOUT) -> +3V3
- U3 pad 1: GND -> GNDA
- U3 pad 4: 3V3 -> +3V3
- U3 pad 5: /SENSOR INPUT/GPIO_18 -> /MCU (page 4)/GPIO_18
- U3 pad 6: /SENSOR INPUT/GPIO_17 -> /MCU (page 4)/GPIO_17
- U3 pad 7: /SENSOR INPUT/GPIO_16 -> /MCU (page 4)/GPIO_16
Routing:
- net GND: track 0.00 -> 358.5 mm, vias 0 -> 14
- net +5v: track 0.00 -> 244.5 mm, vias 0 -> 2
- net /HV_INPUT + PROTECTION/L_FUSED: track 0.00 -> 193.3 mm, vias 0 -> 1
- net /HV_INPUT + PROTECTION/N_FUSED: track 0.00 -> 133.7 mm
- net /MCU (page 4)/GPIO_10: track 0.00 -> 130.3 mm, vias 0 -> 3
- net +3V3: track 0.00 -> 111.7 mm, vias 0 -> 4
- net /MCU (page 4)/GPIO_11: track 0.00 -> 91.7 mm, vias 0 -> 5
- net /MCU (page 4)/GPIO_12: track 0.00 -> 90.8 mm, vias 0 -> 3
- net GNDA: track 0.00 -> 68.7 mm, vias 0 -> 2
- net /Relays+RC SNUBBER/3_WAY_VALVE_LOAD: track 0.00 -> 66.2 mm
- net Net-(J23-Pad03): track 0.00 -> 57.5 mm, vias 0 -> 3
- net /Relays+RC SNUBBER/PUMP_LOAD: track 0.00 -> 55.6 mm, vias 0 -> 3
- net /MCU (page 4)/GPIO_20: track 0.00 -> 52.7 mm, vias 0 -> 3
- net /SENSOR INPUT/T+: track 0.00 -> 51.4 mm, vias 0 -> 6
- net /SENSOR INPUT/T-: track 0.00 -> 48.8 mm, vias 0 -> 4
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Other:
- board size 119.4 x 113.1 mm -> 136.6 x 80 mm

Commit message: Update KiCad project files
Parts:
- removed J25: MTLW-104-X-X-S-X, 4 PIN:SAMTEC_MTLW-104-X-X-S-X
- removed J27, J4: Screw_Terminal_01x02, TerminalBlock_Phoenix:TerminalBlock_Phoenix_MKDS-1,5-2-5.08_1x02_P5.08mm_Horizontal
- removed J3: Screw_Terminal_01x02, TerminalBlock_Phoenix:TerminalBlock_Phoenix_MKDS-3-2-5.08_1x02_P5.08mm_Horizontal
- removed J5: Screw_Terminal_01x03, TerminalBlock_Phoenix:TerminalBlock_Phoenix_MKDS-1,5-3-5.08_1x03_P5.08mm_Horizontal
- added J13: 1725740, 11 PIN:PHOENIX_1725740, F.Cu at (210.7, 93.3)
- J2: value Screw_Terminal_01x02 -> Screw_Terminal_01x04; footprint TerminalBlock_Phoenix:TerminalBlock_Phoenix_MKDS-3-2-5.08_1x02_P5.08mm_Horizontal -> TerminalBlock_TE-Connectivity:TerminalBlock_TE_282834-4_1x04_P2.54mm_Horizontal
- P1: moved to F.Cu
- moved J2 115.9 mm to (76.9, 41.1), turned to 0 degrees
- moved J26 34.2 mm to (209.2, 62.0)
- moved J20 30.0 mm to (198.6, 44.9)
- moved D10 23.9 mm to (198.4, 63.6)
- moved J24 22.6 mm to (200.8, 87.3)
- moved J19 14.6 mm to (186.7, 44.9)
- moved J17 13.6 mm to (192.7, 44.9)
- moved R21 12.7 mm to (202.0, 66.4), turned to 0 degrees
- moved H3 10.4 mm to (201.5, 101.0)
- moved H1 5.39 mm to (83.1, 50.7)
- moved H2 5.39 mm to (203.6, 50.2)
- moved J21 3.83 mm to (168.7, 45.0)
- moved F1 3.23 mm to (79.3, 55.3)
- moved J6 2.70 mm to (88.4, 44.9)
- moved BZ1 2.67 mm to (189.5, 58.3)
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Connections:
- net /SENSOR INPUT/T- renamed THERMOCOUPLE-
- net Net-(D10-A) renamed STEAM_HEATER_-(C)
- D9 pad 2: Net-(D9-A) -> BREW_HEATER_-(C)
- J2 pad 1: +5v -> /HV_INPUT + PROTECTION/L_FUSED
- J2 pad 2: Net-(D9-A) -> /PORTS/CT_LINE_-
- Q5 pad 3: Net-(D9-A) -> BREW_HEATER_-(C)
- R26 pad 1: /SENSOR INPUT/TRANSDUCER_SIGNAL -> PRESSUE-SIGNAL
- TP5 pad 1: /PORTS/GPIO_26 -> /MCU (page 4)/GPIO_26
- TP6 pad 1: /PORTS/GPIO_27 -> /MCU (page 4)/GPIO_27
- TP7 pad 1: /PORTS/GPIO_28 -> /SENSOR INPUT/GPIO_28
- U3 pad 3: /SENSOR INPUT/T+ -> THERMOCOUPLE+
Routing:
- net GND: track 358.5 -> 238.7 mm, vias 14 -> 20
- net /MCU (page 4)/GPIO_11: track 91.7 -> 0.00 mm, vias 5 -> 0
- net /SENSOR INPUT/T+: track 51.4 -> 0.00 mm, vias 6 -> 0
- net THERMOCOUPLE-: track 48.8 -> 3.06 mm, vias 4 -> 0
- net Net-(D9-A): track 41.3 -> 0.00 mm, vias 1 -> 0
- net /SENSOR INPUT/TRANSDUCER_SIGNAL: track 28.3 -> 0.00 mm
- net GPIO22: track 38.4 -> 11.8 mm, vias 1 -> 0
- net /HV_INPUT + PROTECTION/N_FUSED: track 133.7 -> 107.2 mm
- net /HV_INPUT + PROTECTION/L_FUSED: track 193.3 -> 170.1 mm
- net Net-(P1-Pad3): track 16.6 -> 0.00 mm
- net BREW_HEATER_-(C): track 0.00 -> 13.3 mm
- net STEAM_HEATER_-(C): track 9.00 -> 19.7 mm, vias 0 -> 2
- net +5v: track 244.5 -> 253.2 mm, vias 2 -> 4
- net THERMOCOUPLE+: track 0.00 -> 7.71 mm
- net /Relays+RC SNUBBER/PUMP_LOAD: track 55.6 -> 49.1 mm, vias 3 -> 1
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- added copper zone on B.Cu, net GND

Commit message: Updated PCB files
Parts:
- removed D5: 1N4007, Diode_SMD:D_SMA
- removed D6: LED, LED_SMD:LED_0805_2012Metric
- removed J1, J10, J11, J14, J15, J16, J17, J18, J19, J20, J21, J22, J6, J7, J8, J9: 928814-1, 6.3mm spade:TE_928814-1
- removed J12: Screw_Terminal_01x03, TerminalBlock_Phoenix:TerminalBlock_Phoenix_MKDS-1,5-3-5.08_1x03_P5.08mm_Horizontal
- removed J13: 1725740, 11 PIN:PHOENIX_1725740
- removed J2: Screw_Terminal_01x04, TerminalBlock_TE-Connectivity:TerminalBlock_TE_282834-4_1x04_P2.54mm_Horizontal
- removed K3: G2RL-1-H, RELAY:Relay_SPDT_Omron_G2RL-1 MODIFIED
- removed Q3: MMBT2222A, Package_TO_SOT_SMD:SOT-23
- removed R12: 10K, Resistor_SMD:R_0805_2012Metric
- removed R8: 1K, Resistor_SMD:R_0805_2012Metric
- removed R9: 470, Resistor_SMD:R_0805_2012Metric
- removed TP1, TP2, TP3: TestPoint_Alt, Connector_Pin:Pin_D1.0mm_L10.0mm_LooseFit
- added 5V801: TestPoint_Alt, Connector_Pin:Pin_D1.0mm_L10.0mm_LooseFit, F.Cu at (150.4, 72.4)
- added ADC_REF801: TestPoint_Alt, Connector_Pin:Pin_D1.0mm_L10.0mm_LooseFit, F.Cu at (160.7, 105.6)
- added GND801: TestPoint_Alt, Connector_Pin:Pin_D1.0mm_L10.0mm_LooseFit, F.Cu at (144.4, 96.8)
- added J201: 928814-1, 6.3mm spade:TE_928814-1, F.Cu at (92.1, 44.7)
- added J202: 928814-1, 6.3mm spade:TE_928814-1, F.Cu at (127.4, 44.7)
- added J203: 928814-1, 6.3mm spade:TE_928814-1, F.Cu at (100.1, 44.7)
- added J204: 928814-1, 6.3mm spade:TE_928814-1, F.Cu at (139.2, 44.7)
- added J206: 928814-1, 6.3mm spade:TE_928814-1, F.Cu at (115.6, 44.7)
- added J209: 928814-1, 6.3mm spade:TE_928814-1, F.Cu at (108.0, 44.7)
- added J702: Screw_Terminal_01x06, TerminalBlock_Phoenix:TerminalBlock_Phoenix_MPT-0,5-6-2.54_1x06_P2.54mm_Horizontal, F.Cu at (207.3, 59.4)
- added J703: Screw_Terminal_01x12, TerminalBlock_Phoenix:TerminalBlock_Phoenix_MPT-0,5-12-2.54_1x12_P2.54mm_Horizontal, F.Cu at (207.4, 91.6)
- added J801: MTLW-104-X-X-S-X, 4 PIN:SAMTEC_MTLW-104-X-X-S-X, F.Cu at (81.3, 40.2)
- C10, C11, C7, R49: moved to B.Cu
- D10, D3, D4, D8, D9: moved to F.Cu
- moved IO26 92.3 mm to (161.0, 93.0)
- moved IO27 91.2 mm to (161.7, 88.7)
- moved C9 82.9 mm to (167.4, 104.6), turned to -90 degrees
- moved D16 82.4 mm to (175.2, 46.1), turned to 180 degrees
- moved D3 72.1 mm to (168.0, 46.1), turned to 0 degrees
- moved FB1 70.6 mm to (163.9, 105.2), turned to 90 degrees
- moved C11 61.5 mm to (183.9, 66.2), turned to 180 degrees
- moved R49 60.8 mm to (178.7, 73.8), turned to 90 degrees
- moved D4 60.6 mm to (160.6, 46.1)
- moved R15 58.2 mm to (200.8, 107.6), turned to -90 degrees
- moved D8 56.4 mm to (164.3, 46.1), turned to 180 degrees
- moved C7 51.1 mm to (188.4, 67.2), turned to 180 degrees
- moved C10 47.5 mm to (201.8, 63.3), turned to 180 degrees
- moved R48 38.7 mm to (198.4, 63.6)
- moved D9 35.8 mm to (183.0, 45.0)
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- renumbered TP4 to 3V3, TP5 to IO26, TP6 to IO27, TP7 to IO28
Connections:
- net /HV_INPUT + PROTECTION/LIVE renamed Net-(F1-Pad1)
- net /Relays+RC SNUBBER/3_WAY_VALVE_LOAD renamed 3_WAY_VALVE_LOAD
- net /Relays+RC SNUBBER/PUMP_LOAD renamed PUMP_LOAD
- A1 pad 26: /MCU (page 4)/GPIO_20 -> unconnected-(A1-GPIO20-Pad26)
- K2 pad 14: /Relays+RC SNUBBER/LED_LOAD -> LED_LOAD
Routing:
- net CT_LINE-: track 0.00 -> 158.2 mm, vias 0 -> 1
- net CT_LINE+: track 0.00 -> 157.0 mm, vias 0 -> 3
- net PIN_RUN: track 11.3 -> 108.4 mm, vias 1 -> 10
- net /MCU (page 4)/GPIO_2: track 27.5 -> 116.9 mm, vias 1 -> 4
- net Net-(D3-K): track 1.84 -> 89.9 mm, vias 0 -> 3
- net +5v: track 253.2 -> 337.0 mm, vias 4 -> 7
- net Net-(D1-A): track 27.2 -> 106.9 mm, vias 1 -> 2
- net /SENSOR INPUT/AC_OUT: track 0.00 -> 79.6 mm, vias 0 -> 11
- net THERMOCOUPLE-: track 3.06 -> 75.7 mm, vias 0 -> 6
- net B00T_SEL: track 10.4 -> 80.3 mm, vias 1 -> 5
- net Net-(D8-K): track 2.09 -> 70.9 mm, vias 0 -> 5
- net /MCU (page 4)/GPIO_11: track 0.00 -> 65.5 mm, vias 0 -> 9
- net /MCU (page 4)/GPIO_3: track 35.3 -> 100.5 mm, vias 3 -> 8
- net THERMOCOUPLE+: track 7.71 -> 72.5 mm, vias 0 -> 6
- net Net-(D4-K): track 2.98 -> 67.0 mm, vias 0 -> 5
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Other:
- board text added: "3V3"
- board text added: "5v"
- board text added: "AC"
- board text added: "ADC_REF"
- board text added: "BREW"
- board text added: "CT+"
- board text added: "CT-"
- board text added: "DEBUG"
- board text added: "EARTH"
- board text added: "GND"
- board text added: "IO0"
- board text added: "IO1"
- board text added: "IO2"
- board text added: "IO3"
- board text added: "IO5"
- board text added: "IO6"
- board text added: "IO7"
- board text added: "IO8"
- board text added: "IO9"
- board text added: "LED"
- board text added: "LIVE"
- board text added: "N"
- board text added: "POWERMETER"
- board text added: "PSI"
- board text added: "PUMP"
- board text added: "STEAM"
- board text added: "T+"
- board text added: "T-"
- board text added: "VALVE"
