File: ECM Synchronika Custom Control Board.kicad_pcb (KiCad board)
At the start: 2 copper layers, 136.6 x 80 mm, 133 parts, among them J201 928814-1, J202 928814-1, J203 928814-1, J204 928814-1, J206 928814-1, J209 928814-1, J23 MTLW-104-X-X-S-X, J24 MTLW-104-X-X-S-X, J26 TSW-105-05-L-S-LL, J702 Screw_Terminal_01x06, J703 Screw_Terminal_01x12, J801 MTLW-104-X-X-S-X, K1 G2RL-1-H, K2 G2RL-1-H, K4 G2RL-1-H, P1 BM08B-GHS-TBT_LF__SN__N_, Q1 MMBT2222A, Q2 MMBT2222A, Q4 MMBT2222A, Q5 MMBT2222A, Q6 MMBT2222A, SW1 SW_Push, SW2 SW_Push, U1 AP2112K-3.3, U3 MAX31855KASA, U4 OPA342UA, U5 TLV3201AIDBVR

Commit message: Updated PCB files
Parts:
- moved D9 4.26 mm to (178.9, 46.1)
Routing:
- net Net-(D9-K): track 42.5 -> 43.6 mm
- net BREW_HEATER_-(C): track 54.1 -> 55.1 mm
Other:
- board text added: "I2C"
- board text added: "LV METER"
Changed lines of the file:
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@@
 		(tags "LED")
 		(property "Reference" "D8"
-			(at -0.64 2.06 0)
+			(at -0.05 1.64 0)
 			(layer "F.SilkS")
 			(effects
@@
 		(tags "tact sw push 6mm")
 		(property "Reference" "SW2"
-			(at 3.25 -2 90)
+			(at -2.57 1.4 180)
 			(layer "F.SilkS")
 			(effects
@@
 			(at 0 -3.7 0)
 			(layer "F.SilkS")
+			(hide yes)
 			(effects
 				(font
@@
 			(at 0 -3.7 0)
 			(layer "F.SilkS")
+			(hide yes)
 			(effects
 				(font
@@
 		(tags "LED")
 		(property "Reference" "D3"
-			(at -0.75 -1.63 0)
+			(at -0.2 -1.61 0)
 			(layer "F.SilkS")
 			(effects
@@
 		(tags "tact sw push 6mm")
 		(property "Reference" "SW1"
-			(at 8.71 -1.94 180)
+			(at -2.28 1.46 180)
 			(layer "F.SilkS")
 			(effects
@@
 		(tags "THT Terminal Block Phoenix MPT-0,5-12-2.54 pitch 2.54mm size 30.9x6.2mm drill 1.1mm pad 2.2mm")
 		(property "Reference" "J703"
-			(at -2.59 -5.54 180)
+			(at 14.83 -8.44 270)
 			(layer "F.SilkS")
 			(effects
@@
 	(footprint "LED_SMD:LED_0805_2012Metric"
 		(layer "F.Cu")
-		(at 183.0325 45.02 180)
+		(at 178.9075 46.07 180)
 		(descr "LED SMD 0805 (2012 Metric), square (rectangular) end terminal, IPC-7351 nominal, (Body size source: https://docs.google.com/spreadsheets/d/1BsfQQcO9C6DZCsRaXUlFlo91Tg2WpOkGARC1WS5S8t0/edit?usp=sharing), generated with kicad-footprint-generator")
 		(tags "LED")
 		(property "Reference" "D9"
-			(at -0.3425 1.89 0)
+			(at -0.1825 1.62 0)
 			(layer "F.SilkS")
 			(effects
@@
 		)
 	)
+	(gr_text "LV METER\n	"
+		(at 192.69 43.61 270)
+		(layer "F.SilkS")
+		(effects
+			(font
+				(size 1 1)
+				(thickness 0.1)
+			)
+			(justify left bottom)
+		)
+	)
 	(gr_text "GND"
 		(at 202.51 55.55 270)
@@
 		)
 	)
+	(gr_text "I2C"
+		(at 197.02 88.82 90)
+		(layer "F.SilkS")
+		(effects
+			(font
+				(size 1 1)
+				(thickness 0.1)
+			)
+			(justify left bottom)
+		)
+	)
 	(gr_text "IO5"
 		(at 201.48 60.75 0)
@@
 	)
 	(segment
+		(start 179.906 46.009)
+		(end 179.845 46.07)
+		(width 0.3)
+		(layer "F.Cu")
+		(net 10)
+	)
+	(segment
 		(start 193.369 56.509)
 		(end 191.97 55.11)
@@
 	)
 	(segment
+		(start 182.74 45.91)
+		(end 182.0725 45.91)
+		(width 0.3)
+		(layer "F.Cu")
+		(net 10)
+	)
+	(segment
 		(start 190.38 54.01)
 		(end 185.82 49.45)
@@
 	)
 	(segment
+		(start 182.0725 45.91)
+		(end 181.9735 46.009)
+		(width 0.3)
+		(layer "F.Cu")
+		(net 10)
+	)
+	(segment
 		(start 191.97 55.05)
 		(end 191.93 55.01)
@@
 	)
 	(segment
-		(start 183.9 44.95)
-		(end 183.97 45.02)
+		(start 181.9735 46.009)
+		(end 179.906 46.009)
 		(width 0.3)
 		(layer "F.Cu")
@@
 	)
 	(segment
-		(start 183.0325 44.95)
-		(end 183.9 44.95)
-		(width 0.3)
-		(layer "F.Cu")
-		(net 10)
-	)
-	(segment
 		(start 200.5 68.19)
 		(end 195.49 63.18)
@@
 	)
 	(via
-		(at 183.0325 44.95)
+		(at 182.74 45.91)
 		(size 0.5)
 		(drill 0.3)
@@
 	)
 	(segment
-		(start 185.47 49.45)
-		(end 183.0325 47.0125)
+		(start 190.93 54.01)
+		(end 190.38 54.01)
 		(width 0.3)
 		(layer "B.Cu")
@@
 	)
 	(segment
-		(start 190.93 54.01)
-		(end 190.38 54.01)
+		(start 183.0325 46.2025)
+		(end 183.0325 47.0125)
 		(width 0.3)
 		(layer "B.Cu")
@@
 	)
 	(segment
+		(start 182.74 45.91)
+		(end 183.0325 46.2025)
+		(width 0.3)
+		(layer "B.Cu")
+		(net 10)
+	)
+	(segment
 		(start 201.03 76.22)
 		(end 200.5 75.69)
@@
 	)
 	(segment
-		(start 185.6 49.45)
-		(end 185.47 49.45)
+		(start 185.47 49.45)
+		(end 185.6 49.45)
 		(width 0.3)
 		(layer "B.Cu")
@@
 	(segment
 		(start 183.0325 47.0125)
-		(end 183.0325 44.95)
+		(end 185.47 49.45)
 		(width 0.3)
 		(layer "B.Cu")
@@
 	(segment
 		(start 178.57 44.54)
-		(end 171.97 44.54)
+		(end 178.32 44.54)
 		(width 0.3)
 		(layer "F.Cu")
@@
 	)
 	(segment
+		(start 178.32 44.54)
+		(end 171.97 44.54)
+		(width 0.3)
+		(layer "F.Cu")
+		(net 11)
+	)
+	(segment
 		(start 201.370058 66.25)
 		(end 200.34 65.219942)
@@
 	)
 	(segment
-		(start 202.059 66.25)
-		(end 201.370058 66.25)
+		(start 178.341 44.519)
+		(end 178.32 44.54)
 		(width 0.3)
 		(layer "F.Cu")
@@
 	)
 	(segment
-		(start 180.54 46.51)
-		(end 178.57 44.54)
+		(start 182.889 44.519)
+		(end 178.341 44.519)
 		(width 0.3)
 		(layer "F.Cu")
@@
 	(segment
 		(start 184.88 46.51)
-		(end 180.54 46.51)
+		(end 182.889 44.519)
+		(width 0.3)
+		(layer "F.Cu")
+		(net 11)
+	)
+	(segment
+		(start 202.059 66.25)
+		(end 201.370058 66.25)
 		(width 0.3)
 		(layer "F.Cu")
@@
 	)
 	(segment
+		(start 179.02 45.02)
+		(end 177.97 46.07)
+		(width 0.3)
+		(layer "F.Cu")
+		(net 68)
+	)
+	(segment
 		(start 195.29 71.39)
 		(end 195 71.1)
@@
 	)
 	(segment
+		(start 181.51 45.26)
+		(end 181.27 45.02)
+		(width 0.3)
+		(layer "F.Cu")
+		(net 68)
+	)
+	(segment
 		(start 192.149 59.061)
 		(end 192.149 57.239)
@@
 	)
 	(segment
-		(start 192.149 57.239)
-		(end 191.84 56.93)
+		(start 181.27 45.02)
+		(end 179.02 45.02)
 		(width 0.3)
 		(layer "F.Cu")
@@
 	)
 	(segment
-		(start 188.74 53.72)
-		(end 188.54 53.72)
+		(start 192.149 57.239)
+		(end 191.84 56.93)
 		(width 0.3)
 		(layer "F.Cu")
@@
 	)
 	(segment
-		(start 182.04 43.53)
-		(end 182.04 44.965)
+		(start 188.74 53.72)
+		(end 188.54 53.72)
 		(width 0.3)
 		(layer "F.Cu")
@@
 		(net 68)
 	)
-	(segment
-		(start 182.04 44.965)
-		(end 182.095 45.02)
-		(width 0.3)
-		(layer "F.Cu")
-		(net 68)
-	)
 	(via
 		(at 195 71.1)
@@
 	)
 	(via
-		(at 182.04 43.53)
+		(at 195.273191 69.421553)
 		(size 0.5)
 		(drill 0.3)
@@
 	)
 	(via
-		(at 195.273191 69.421553)
+		(at 192.149 59.061)
 		(size 0.5)
 		(drill 0.3)
@@
 	)
 	(via
-		(at 192.149 59.061)
+		(at 195.23 75.88)
 		(size 0.5)
 		(drill 0.3)
@@
 	)
 	(via
-		(at 195.23 75.88)
+		(at 191.84 56.93)
 		(size 0.5)
 		(drill 0.3)
@@
 	)
 	(via
-		(at 191.84 56.93)
+		(at 194.670735 64.879265)
 		(size 0.5)
 		(drill 0.3)
@@
 	)
 	(via
-		(at 194.670735 64.879265)
+		(at 181.51 45.26)
 		(size 0.5)
 		(drill 0.3)
@@
 	)
 	(segment
+		(start 182.04 45.79)
+		(end 182.04 47.15)
+		(width 0.3)
+		(layer "B.Cu")
+		(net 68)
+	)
+	(segment
 		(start 198.88 76.74)
 		(end 198.87 76.75)
@@
 	)
 	(segment
-		(start 182.04 47.15)
-		(end 182.04 43.53)
+		(start 198.87 76.75)
+		(end 195.7425 76.75)
 		(width 0.3)
 		(layer "B.Cu")
@@
 	)
 	(segment
-		(start 198.87 76.75)
-		(end 195.7425 76.75)
+		(start 205.42 79.1)
+		(end 202.4825 79.1)
 		(width 0.3)
 		(layer "B.Cu")
@@
 	)
 	(segment
-		(start 205.42 79.1)
-		(end 202.4825 79.1)
+		(start 181.51 45.26)
+		(end 182.04 45.79)
 		(width 0.3)
 		(layer "B.Cu")
@@
 	)
 	(segment
-		(start 184.98 50.09)
-		(end 182.04 47.15)
+		(start 182.04 47.15)
+		(end 184.98 50.09)
 		(width 0.3)
 		(layer "B.Cu")
