File: PORTS.kicad_sch (KiCad schematic)
At the start: 16 parts, among them J23 MTLW-104-X-X-S-X, J24 MTLW-104-X-X-S-X, J25 MTLW-104-X-X-S-X, J26 TSW-105-05-L-S-LL, J27 Screw_Terminal_01x02, P1 BM08B-GHS-TBT_LF__SN__N_

Commit message: Update KiCad project files
Connections:
- net GPIO0: now also R44.2
Other:
- note added: "DEBUG PORT"
- note added: "ESP32 DISPLAY MODULE INTERFACE"
- note added: "I2C ACCESSORY PORT"
- note added: "Power Metering"
- moved on the sheet: J23, J24, J25, J26, J27, R44, R45, R46, R47

Commit message: Update KiCad project files
Parts:
- added TP1, TP2, TP3, TP4, TP5, TP6, TP7: TestPoint_Alt, Connector_Pin:Pin_D1.0mm_L10.0mm_LooseFit, symbol Connector:TestPoint_Alt
- J23, J24, J25: footprint MTLW-104-X-X-S-X:SAMTEC_MTLW-104-X-X-S-X -> 4 PIN:SAMTEC_MTLW-104-X-X-S-X
- J26: footprint TSW-105-05-L-S-LL:SAMTEC_TSW-105-05-L-S-LL -> 5 PIN:SAMTEC_TSW-105-05-L-S-LL
- P1: footprint BM08B-GHS-TBT_LF__SN__N_:JST_BM08B-GHS-TBT_LF__SN__N_ -> 8 PIN HEADER:JST_BM08B-GHS-TBT_LF__SN__N_
Connections:
- net +3V3: now also TP4.1
- net +5v: now also TP3.1
- net GND: now also TP1.1
- new net ADC-REF: TP2.1
- new net GPIO_26: TP5.1
- new net GPIO_27: TP6.1
- new net GPIO_28: TP7.1

Commit message: Update KiCad project files
Parts:
- removed J25: MTLW-104-X-X-S-X, 4 PIN:SAMTEC_MTLW-104-X-X-S-X, symbol 4_pin:MTLW-104-X-X-S-X
- removed J27: Screw_Terminal_01x02, TerminalBlock_Phoenix:TerminalBlock_Phoenix_MKDS-1,5-2-5.08_1x02_P5.08mm_Horizontal, symbol Connector:Screw_Terminal_01x02
- added J13: 1725740, 11 PIN:PHOENIX_1725740, symbol 11 PIN:1725740
- added J2: Screw_Terminal_01x04, TerminalBlock_TE-Connectivity:TerminalBlock_TE_282834-4_1x04_P2.54mm_Horizontal, symbol Connector:Screw_Terminal_01x04
Connections:
- net +5v: now also J13.3, J13.7, J13.9
- net CT_LINE_+: now also J13.10, J2.3 (Pin_3)
- net CT_LINE_-: now also J13.11, J2.2 (Pin_2)
- net GND: now also J13.2
- net L_FUSED: now also J2.1 (Pin_1)
- net N_FUSED: now also J2.4 (Pin_4)
- new net BREW_HEATER_-(C): J13.6
- new net PRESSUE-SIGNAL: J13.1
- new net STEAM_HEATER_-(C): J13.8
- new net THERMOCOUPLE+: J13.4
- new net THERMOCOUPLE-: J13.5

Commit message: Updated PCB files
Parts:
- removed J13: 1725740, 11 PIN:PHOENIX_1725740, symbol 11 PIN:1725740
- removed J2: Screw_Terminal_01x04, TerminalBlock_TE-Connectivity:TerminalBlock_TE_282834-4_1x04_P2.54mm_Horizontal, symbol Connector:Screw_Terminal_01x04
- added J801: MTLW-104-X-X-S-X, 4 PIN:SAMTEC_MTLW-104-X-X-S-X, symbol 4_pin:MTLW-104-X-X-S-X
- renumbered TP4 to 3V3, TP3 to 5V, TP2 to ADC_REF, TP1 to GND, TP5 to IO26, TP6 to IO27, TP7 to IO28
Connections:
- net L_FUSED: now also J801.01
- net N_FUSED: now also J801.04
- new net CT_LINE+: J801.03
- new net CT_LINE-: J801.02

Commit message: Updated PCB files
Parts:
- renumbered 5V to 5V801, ADC_REF to ADC_REF801, GND to GND801
Changed lines of the file:
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@@
 		(dnp no)
 		(fields_autoplaced yes)
-		(property "Reference" "ADC_REF"
+		(property "Reference" "ADC_REF801"
 			(at 46.99 177.0379 0)
 			(effects
@@
 			(project "ECM Synchronika Custom Control Board"
 				(path "/0a1cfe74-4adf-4cda-8eff-54fb631bdb34/180ab2c6-997f-4c3b-b693-7bfb58c46537"
-					(reference "ADC_REF")
+					(reference "ADC_REF801")
 					(unit 1)
 				)
@@
 		(dnp no)
 		(fields_autoplaced yes)
-		(property "Reference" "5V"
+		(property "Reference" "5V801"
 			(at 83.82 177.0379 0)
 			(effects
@@
 			(project "ECM Synchronika Custom Control Board"
 				(path "/0a1cfe74-4adf-4cda-8eff-54fb631bdb34/180ab2c6-997f-4c3b-b693-7bfb58c46537"
-					(reference "5V")
+					(reference "5V801")
 					(unit 1)
 				)
@@
 		(dnp no)
 		(fields_autoplaced yes)
-		(property "Reference" "GND"
+		(property "Reference" "GND801"
 			(at 63.5 177.0379 0)
 			(effects
@@
 			(project "ECM Synchronika Custom Control Board"
 				(path "/0a1cfe74-4adf-4cda-8eff-54fb631bdb34/180ab2c6-997f-4c3b-b693-7bfb58c46537"
-					(reference "GND")
-					(unit 1)
-				)
+					(reference "GND801")
+					(unit 1)
+				)
